File: SIM/mixer/mixer.sch (KiCad schematic (older format))
At the start: 12 parts, among them U1 LF356

Commit message: added files to repo
Parts:
- added C1, C2, C3, C4: 10u, symbol pspice:C
- R1: value 40k -> 40K
- R2: value 10k -> 10K
- V1: Spice_Model sin(0 1.5 1k) -> sin(1.5 1.5 8k)
- V2, V3: Spice_Model dc(50) -> dc(4.5)
- V4: Spice_Model sin(0 1.5 2k) -> sin(1.5 1.5 8k)
- V5: Spice_Model sin(0 1.5 4k) -> sin(1.5 1.5 8k)
- V6: Spice_Model sin(0 1.5 8k) -> sin(1.5 1.5 8k)
Connections:
- net IN: now also C1.1; no longer V1.1
- net IN1: now also C2.1; no longer V4.1
- net IN2: now also C3.1; no longer V5.1
- net IN3: now also C4.1; no longer V6.1
- new net: C1.2, V1.1
- new net: C2.2, V4.1
- new net: C3.2, V5.1
- new net: C4.2, V6.1
Other:
- moved on the sheet: V1, V4, V5, V6

Commit message: update
Parts:
- removed C1, C2, C3, C4: 10u, symbol pspice:C
- removed R3, R4, R5: 40k, symbol pspice:R
- removed V4, V5, V6: VSIN, symbol Simulation_SPICE:VSIN
- added C1, C2: 10u, symbol pspice:CAP
- added R2: 100k, symbol pspice:R
- added V2: VSIN, symbol Simulation_SPICE:VSIN
- R1: value 40K -> 100k
- R4: renamed from R2; value 10K -> 50k
- V3: renamed from V2; Spice_Model dc(4.5) -> dc(12)
- V4: renamed from V3; Spice_Model dc(4.5) -> dc(12)
Connections:
- net GND: now also R2.1, V2.2
- net IN: now also V1.1, C2.2; no longer R1.2
- net IN2: now also C1.2, V2.1
- new net: C2.1, R1.2
- new net: C1.1, R2.2
Other:
- moved on the sheet: R1
