File: Hardware/V1_0/V1_0.sch (KiCad schematic (older format))
At the start: 0 parts

Commit message: some work on the MCU part
Parts:
- added C1: 2.2u, Capacitor_SMD:C_0603_1608Metric, symbol Device:C_Small
- added J1: Micro_SD_Card_Det, Connector_Card:microSD_HC_Hirose_DM3D-SF, symbol Connector:Micro_SD_Card_Det
- added R1, R2, R3, R4, R5, R6, R7: 10k, Resistor_SMD:R_0603_1608Metric, symbol Device:R_Small
Connections:
- new net +3V3: C1.1, J1.4 (VDD), R1.2, R2.2, R3.2, R4.2, R5.2, R6.2, R7.2
- new net GND: C1.2, J1.11 (SHIELD), J1.6 (VSS), J1.9 (DET_B)
- new net MCU/SDIO_CK: J1.5 (CLK), R4.1
- new net MCU/SDIO_CMD: J1.3 (CMD), R5.1
- new net MCU/SDIO_D0: J1.7 (DAT0), R3.1
- new net MCU/SDIO_D1: J1.8 (DAT1), R2.1
- new net MCU/SDIO_D2: J1.1 (DAT2), R7.1
- new net MCU/SDIO_D3: J1.2 (DAT3/CD), R6.1
- new net MCU/SDIO_DET: J1.10 (DET_A), R1.1
Other:
- note added: "SD Card for logging,\nsample buffering, etc."

Commit message: tweaks
Other:
- note added: "Waveform storage\n"
- note removed: "SD Card for logging,\nsample buffering, etc."
Changed lines of the file:
@@
 encoding utf-8
 Sheet 1 4
-Title ""
+Title "SYNTH"
 Date ""
-Rev ""
-Comp ""
+Rev "1"
+Comp "Bo Joel Svensson"
 Comment1 ""
 Comment2 ""
@@
 $EndDescr
 $Sheet
-S 4600 3800 1150 1500
+S 2150 5900 1150 1500
 U 5E063F78
 F0 "DCDC" 50
@@
 $EndSheet
 $Sheet
-S 7600 3850 1000 1500
+S 5100 3550 1000 1500
 U 5E06400A
 F0 "Information" 50
@@
 	6950 2350 7000 2350
 Connection ~ 5000 2700
-Text Notes 7600 2500 0    50   ~ 0
-SD Card for logging,\nsample buffering, etc.
 $Sheet
 S 2050 1100 1500 4400
@@
 	3550 2150 4650 2150
 Connection ~ 4650 2150
+Text Notes 5750 2400 0    50   ~ 0
+Waveform storage\n
 $EndSCHEMATC

Commit message: low energy work
Changed lines of the file:
@@
 F0 "DCDC" 50
 F1 "DCDC.sch" 50
-$EndSheet
-$Sheet
-S 5100 3550 1000 1500
-U 5E06400A
-F0 "Information" 50
-F1 "Information.sch" 50
+F2 "VREF" I R 3300 6050 50
+F3 "RAIL-" I R 3300 6300 50
+F4 "RAIL+" I R 3300 6200 50
 $EndSheet
 $Comp
@@
 F10 "SDIO_CMD" I R 3550 1650 50
 F11 "VREF" I L 2050 3200 50
+F12 "HBEN" I R 3550 5300 50
+F13 "DB7" I R 3550 4900 50
+F14 "NWR" I R 3550 5200 50
+F15 "DB2" I R 3550 4400 50
+F16 "NLDAC" I R 3550 5000 50
+F17 "DB5" I R 3550 4700 50
+F18 "DB0" I R 3550 4200 50
+F19 "DB3" I R 3550 4500 50
+F20 "DB6" I R 3550 4800 50
+F21 "DB1" I R 3550 4300 50
+F22 "DB4" I R 3550 4600 50
+F23 "NCLR" I R 3550 5100 50
+F24 "DMUX0" I R 3550 3850 50
+F25 "DMUX1" I R 3550 3950 50
 $EndSheet
 Wire Wire Line
@@
 Text Notes 5750 2400 0    50   ~ 0
 Waveform storage\n
+Wire Wire Line
+	2050 3200 1750 3200
+Wire Wire Line
+	1750 3200 1750 5750
+Wire Wire Line
+	1750 5750 3550 5750
+Wire Wire Line
+	3550 5750 3550 6050
+Wire Wire Line
+	3550 6050 3300 6050
+Connection ~ 3550 5750
+$Sheet
+S 5150 3050 1250 3550
+U 5E06400A
+F0 "DACS" 50
+F1 "Information.sch" 50
+F2 "VREF" I L 5150 5750 50
+F3 "RAIL+" I L 5150 6200 50
+F4 "RAIL-" I L 5150 6300 50
+F5 "DMUX0" I L 5150 3850 50
+F6 "DMUX1" I L 5150 3950 50
+F7 "DB0" I L 5150 4200 50
+F8 "DB1" I L 5150 4300 50
+F9 "DB2" I L 5150 4400 50
+F10 "DB3" I L 5150 4500 50
+F11 "DB4" I L 5150 4600 50
+F12 "DB5" I L 5150 4700 50
+F13 "DB6" I L 5150 4800 50
+F14 "DB7" I L 5150 4900 50
+F15 "NLDAC" I L 5150 5000 50
+F16 "NCLR" I L 5150 5100 50
+F17 "NWR" I L 5150 5200 50
+F18 "HBEN" I L 5150 5300 50
+F19 "DAC1" I L 5150 3150 50
+F20 "DAC2" I L 5150 3250 50
+$EndSheet
+Wire Wire Line
+	3550 5750 5150 5750
+Wire Wire Line
+	3300 6200 5150 6200
+Wire Wire Line
+	3300 6300 5150 6300
+Wire Wire Line
+	3550 4200 5150 4200
+Wire Wire Line
+	3550 4300 5150 4300
+Wire Wire Line
+	3550 4400 5150 4400
+Wire Wire Line
+	3550 4500 5150 4500
+Wire Wire Line
+	3550 4600 5150 4600
+Wire Wire Line
+	3550 4700 5150 4700
+Wire Wire Line
+	3550 4800 5150 4800
+Wire Wire Line
+	3550 4900 5150 4900
+Wire Wire Line
+	3550 5000 5150 5000
+Wire Wire Line
+	3550 5100 5150 5100
+Wire Wire Line
+	3550 5200 5150 5200
+Wire Wire Line
+	3550 5300 5150 5300
+Wire Wire Line
+	3550 3150 5150 3150
+Wire Wire Line
+	3550 3250 5150 3250
+Wire Wire Line
+	3550 3850 5150 3850
+Wire Wire Line
+	3550 3950 5150 3950
 $EndSCHEMATC

Commit message: update
Changed lines of the file:
@@
 F10 "SDIO_CMD" I R 3550 1650 50
 F11 "VREF" I L 2050 3200 50
-F12 "HBEN" I R 3550 5300 50
-F13 "DB7" I R 3550 4900 50
-F14 "NWR" I R 3550 5200 50
-F15 "DB2" I R 3550 4400 50
-F16 "NLDAC" I R 3550 5000 50
-F17 "DB5" I R 3550 4700 50
-F18 "DB0" I R 3550 4200 50
-F19 "DB3" I R 3550 4500 50
-F20 "DB6" I R 3550 4800 50
-F21 "DB1" I R 3550 4300 50
-F22 "DB4" I R 3550 4600 50
-F23 "NCLR" I R 3550 5100 50
-F24 "DMUX0" I R 3550 3850 50
-F25 "DMUX1" I R 3550 3950 50
+F12 "DB7" I R 3550 4900 50
+F13 "DB2" I R 3550 4400 50
+F14 "DB5" I R 3550 4700 50
+F15 "DB0" I R 3550 4200 50
+F16 "DB3" I R 3550 4500 50
+F17 "DB6" I R 3550 4800 50
+F18 "DB1" I R 3550 4300 50
+F19 "DB4" I R 3550 4600 50
+F20 "N_CLR_0" I R 3550 3500 50
+F21 "N_LDAC_0" I R 3550 3400 50
+F22 "N_WR_0" I R 3550 3600 50
+F23 "BUF_0" I R 3550 3700 50
 $EndSheet
 Wire Wire Line
@@
 	3550 6050 3300 6050
 Connection ~ 3550 5750
-$Sheet
-S 5150 3050 1250 3550
-U 5E06400A
-F0 "DACS" 50
-F1 "Information.sch" 50
-F2 "VREF" I L 5150 5750 50
-F3 "RAIL+" I L 5150 6200 50
-F4 "RAIL-" I L 5150 6300 50
-F5 "DMUX0" I L 5150 3850 50
-F6 "DMUX1" I L 5150 3950 50
-F7 "DB0" I L 5150 4200 50
-F8 "DB1" I L 5150 4300 50
-F9 "DB2" I L 5150 4400 50
-F10 "DB3" I L 5150 4500 50
-F11 "DB4" I L 5150 4600 50
-F12 "DB5" I L 5150 4700 50
-F13 "DB6" I L 5150 4800 50
-F14 "DB7" I L 5150 4900 50
-F15 "NLDAC" I L 5150 5000 50
-F16 "NCLR" I L 5150 5100 50
-F17 "NWR" I L 5150 5200 50
-F18 "HBEN" I L 5150 5300 50
-F19 "DAC1" I L 5150 3150 50
-F20 "DAC2" I L 5150 3250 50
-$EndSheet
 Wire Wire Line
 	3550 5750 5150 5750
@@
 	3550 4900 5150 4900
 Wire Wire Line
-	3550 5000 5150 5000
-Wire Wire Line
-	3550 5100 5150 5100
-Wire Wire Line
-	3550 5200 5150 5200
-Wire Wire Line
-	3550 5300 5150 5300
-Wire Wire Line
 	3550 3150 5150 3150
 Wire Wire Line
 	3550 3250 5150 3250
+$Sheet
+S 5150 3050 1250 3550
+U 5E06400A
+F0 "DACS" 50
+F1 "Information.sch" 50
+F2 "VREF" I L 5150 5750 50
+F3 "RAIL+" I L 5150 6200 50
+F4 "RAIL-" I L 5150 6300 50
+F5 "DB0" I L 5150 4200 50
+F6 "DB1" I L 5150 4300 50
+F7 "DB2" I L 5150 4400 50
+F8 "DB3" I L 5150 4500 50
+F9 "DB4" I L 5150 4600 50
+F10 "DB5" I L 5150 4700 50
+F11 "DB6" I L 5150 4800 50
+F12 "DB7" I L 5150 4900 50
+F13 "DAC1" I L 5150 3150 50
+F14 "DAC2" I L 5150 3250 50
+F15 "N_LDAC_0" I L 5150 3400 50
+F16 "N_CLR_0" I L 5150 3500 50
+F17 "N_WR_0" I L 5150 3600 50
+F18 "BUF_0" I L 5150 3700 50
+$EndSheet
 Wire Wire Line
-	3550 3850 5150 3850
+	3550 3400 5150 3400
 Wire Wire Line
-	3550 3950 5150 3950
+	3550 3500 5150 3500
+Wire Wire Line
+	3550 3600 5150 3600
+Wire Wire Line
+	3550 3700 5150 3700
 $EndSCHEMATC

Commit message: experimenting
Parts:
- added MK1, MK2, MK3, MK4: Mounting_Hole, MountingHole:MountingHole_3.2mm_M3, symbol Mechanical:MountingHole
Changed lines of the file:
@@
 Wire Wire Line
 	3550 3700 5150 3700
+$Comp
+L Mechanical:MountingHole MK2
+U 1 1 5B441268
+P 9300 5900
+F 0 "MK2" H 9400 5946 50  0000 L CNN
+F 1 "Mounting_Hole" H 9400 5855 50  0000 L CNN
+F 2 "MountingHole:MountingHole_3.2mm_M3" H 9300 5900 50  0001 C CNN
+F 3 "" H 9300 5900 50  0001 C CNN
+	1    9300 5900
+	1    0    0    -1
+$EndComp
+$Comp
+L Mechanical:MountingHole MK1
+U 1 1 5B441276
+P 9300 5200
+F 0 "MK1" H 9400 5246 50  0000 L CNN
+F 1 "Mounting_Hole" H 9400 5155 50  0000 L CNN
+F 2 "MountingHole:MountingHole_3.2mm_M3" H 9300 5200 50  0001 C CNN
+F 3 "" H 9300 5200 50  0001 C CNN
+	1    9300 5200
+	1    0    0    -1
+$EndComp
+$Comp
+L Mechanical:MountingHole MK3
+U 1 1 5B44126F
+P 10100 5200
+F 0 "MK3" H 10200 5246 50  0000 L CNN
+F 1 "Mounting_Hole" H 10200 5155 50  0000 L CNN
+F 2 "MountingHole:MountingHole_3.2mm_M3" H 10100 5200 50  0001 C CNN
+F 3 "" H 10100 5200 50  0001 C CNN
+	1    10100 5200
+	1    0    0    -1
+$EndComp
+$Comp
+L Mechanical:MountingHole MK4
+U 1 1 5B441261
+P 10100 5950
+F 0 "MK4" H 10200 5996 50  0000 L CNN
+F 1 "Mounting_Hole" H 10200 5905 50  0000 L CNN
+F 2 "MountingHole:MountingHole_3.2mm_M3" H 10100 5950 50  0001 C CNN
+F 3 "" H 10100 5950 50  0001 C CNN
+	1    10100 5950
+	1    0    0    -1
+$EndComp
 $EndSCHEMATC
