File: Hardware/V1_0/DCDC.sch (KiCad schematic (older format))
At the start: 18 parts, among them U13 MCP16311_2, U7 LM27762

Commit message: some work on the MCU part
Parts:
- R12: renamed from R2; value 285k -> 249k
- R14: renamed from R3; value 90k -> 91k
- renumbered C17 to C14, C19 to C15, C1 to C16, C2 to C17, C21 to C18, C23 to C19, C25 to C20, C3 to C21, C4 to C22, C5 to C23, R1 to R10, R6 to R11, R8 to R13, U7 to U2, U13 to U3
Other:
- note added: "1,2× ((249+91)÷91) = 4.48"
- note added: "−1,22×((249+91)÷91) = −4.56"
- note removed: "1,2× ((285+90)÷90) = 5"
- note removed: "−1,22×((285+90)÷90) = −5,083333333"
Changed lines of the file:
@@
 $EndDescr
 $Comp
-L Regulator_SwitchedCapacitor:LM27762 U7
+L Regulator_SwitchedCapacitor:LM27762 U2
 U 1 1 5E08DC2A
 P 5050 4550
-F 0 "U7" H 5100 5017 50  0000 C CNN
+F 0 "U2" H 5100 5017 50  0000 C CNN
 F 1 "LM27762" H 5100 4926 50  0000 C CNN
 F 2 "Package_SON:WSON-12-1EP_3x2mm_P0.5mm_EP1x2.65_ThermalVias" H 5200 3800 50  0001 L CNN
@@
 Connection ~ 6650 2100
 $Comp
-L Device:C_Small C17
+L Device:C_Small C14
 U 1 1 5B1BFD5B
 P 6500 2350
-F 0 "C17" H 6525 2450 50  0000 L CNN
+F 0 "C14" H 6525 2450 50  0000 L CNN
 F 1 "2.2u" H 6525 2250 50  0000 L CNN
 F 2 "Capacitor_SMD:C_0603_1608Metric" H 6538 2200 30  0001 C CNN
@@
 $EndComp
 $Comp
-L Device:C_Small C19
+L Device:C_Small C15
 U 1 1 5B1BFD62
 P 6750 2350
-F 0 "C19" H 6775 2450 50  0000 L CNN
+F 0 "C15" H 6775 2450 50  0000 L CNN
 F 1 "2.2u" H 6775 2250 50  0000 L CNN
 F 2 "Capacitor_SMD:C_0603_1608Metric" H 6788 2200 30  0001 C CNN
@@
 $EndComp
 $Comp
-L Device:C_Small C23
+L Device:C_Small C19
 U 1 1 5B1BFD69
 P 9000 2350
-F 0 "C23" H 9025 2450 50  0000 L CNN
+F 0 "C19" H 9025 2450 50  0000 L CNN
 F 1 "2.2u" H 9025 2250 50  0000 L CNN
 F 2 "Capacitor_SMD:C_0603_1608Metric" H 9038 2200 30  0001 C CNN
@@
 $EndComp
 $Comp
-L Device:CP1_Small C25
+L Device:CP1_Small C20
 U 1 1 5B1BFD70
 P 9250 2350
-F 0 "C25" H 9275 2450 50  0000 L CNN
+F 0 "C20" H 9275 2450 50  0000 L CNN
 F 1 "100u" H 9275 2250 50  0000 L CNN
 F 2 "Capacitor_Tantalum_SMD:CP_EIA-3528-12_Kemet-T" H 9250 2350 60  0001 C CNN
@@
 $EndComp
 $Comp
-L power:GND #PWR030
+L power:GND #PWR023
 U 1 1 5B1BFD77
 P 8200 2700
-F 0 "#PWR030" H 8200 2450 50  0001 C CNN
+F 0 "#PWR023" H 8200 2450 50  0001 C CNN
 F 1 "GND" H 8200 2550 50  0000 C CNN
 F 2 "" H 8200 2700 60  0000 C CNN
@@
 $EndComp
 $Comp
-L Device:C_Small C21
+L Device:C_Small C18
 U 1 1 5B1BFD7D
 P 8500 1750
-F 0 "C21" H 8525 1850 50  0000 L CNN
+F 0 "C18" H 8525 1850 50  0000 L CNN
 F 1 "100n" H 8525 1650 50  0000 L CNN
 F 2 "Capacitor_SMD:C_0603_1608Metric" H 8538 1600 30  0001 C CNN
@@
 $EndComp
 $Comp
-L Device:R_Small R8
+L Device:R_Small R13
 U 1 1 5B1BFD84
 P 7800 1450
-F 0 "R8" V 7880 1450 50  0000 C CNN
+F 0 "R13" V 7880 1450 50  0000 C CNN
 F 1 "10k" V 7700 1450 50  0000 C CNN
 F 2 "Resistor_SMD:R_0603_1608Metric" V 7730 1450 30  0001 C CNN
@@
 $EndComp
 $Comp
-L Device:R_Small R6
+L Device:R_Small R11
 U 1 1 5B1BFD8B
 P 7100 1450
-F 0 "R6" V 7180 1450 50  0000 C CNN
+F 0 "R11" V 7180 1450 50  0000 C CNN
 F 1 "33k" V 7000 1450 50  0000 C CNN
 F 2 "Resistor_SMD:R_0603_1608Metric" V 7030 1450 30  0001 C CNN
@@
 	6750 2450 6750 2600
 $Comp
-L power:+5V #PWR0107
+L power:+5V #PWR022
 U 1 1 5DD19B4C
 P 6500 1700
-F 0 "#PWR0107" H 6500 1550 50  0001 C CNN
+F 0 "#PWR022" H 6500 1550 50  0001 C CNN
 F 1 "+5V" H 6515 1873 50  0000 C CNN
 F 2 "" H 6500 1700 50  0001 C CNN
@@
 $EndComp
 $Comp
-L power:+3V3 #PWR0103
-U 1 1 5E094974
+L power:+3V3 #PWR024
+U 1 1 5E0CE9A5
 P 9050 1650
-F 0 "#PWR0103" H 9050 1500 50  0001 C CNN
+F 0 "#PWR024" H 9050 1500 50  0001 C CNN
 F 1 "+3V3" H 9065 1823 50  0000 C CNN
 F 2 "" H 9050 1650 50  0001 C CNN
@@
 $EndComp
 $Comp
-L Device:R_Small R2
+L Device:R_Small R12
 U 1 1 5E09D6EB
 P 7650 5900
-F 0 "R2" H 7709 5946 50  0000 L CNN
-F 1 "285k" H 7709 5855 50  0000 L CNN
+F 0 "R12" H 7709 5946 50  0000 L CNN
+F 1 "249k" H 7709 5855 50  0000 L CNN
 F 2 "Resistor_SMD:R_0603_1608Metric" H 7650 5900 50  0001 C CNN
 F 3 "~" H 7650 5900 50  0001 C CNN
@@
 $EndComp
 $Comp
-L Device:R_Small R3
+L Device:R_Small R14
 U 1 1 5E09DEAD
 P 8100 5900
-F 0 "R3" H 8159 5946 50  0000 L CNN
-F 1 "90k" H 8159 5855 50  0000 L CNN
+F 0 "R14" H 8159 5946 50  0000 L CNN
+F 1 "91k" H 8159 5855 50  0000 L CNN
 F 2 "Resistor_SMD:R_0603_1608Metric" H 8100 5900 50  0001 C CNN
 F 3 "~" H 8100 5900 50  0001 C CNN
@@
 $EndComp
 Text Notes 7900 5600 0    50   ~ 0
-1,2× ((285+90)÷90) = 5
+1,2× ((249+91)÷91) = 4.48
 Text Notes 7800 5750 0    50   ~ 0
-−1,22×((285+90)÷90) = −5,083333333
+−1,22×((249+91)÷91) = −4.56
 $Bitmap
 Pos 8500 4650
@@
 $EndBitmap
 $Comp
-L Device:R_Small R1
+L Device:R_Small R10
 U 1 1 5E0A2CA8
 P 6950 4400
-F 0 "R1" H 6891 4446 50  0000 R CNN
+F 0 "R10" H 6891 4446 50  0000 R CNN
 F 1 "10k" H 6891 4355 50  0000 R CNN
 F 2 "Resistor_SMD:R_0603_1608Metric" H 6950 4400 50  0001 C CNN
@@
 $EndComp
 $Comp
-L Device:C_Small C1
+L Device:C_Small C16
 U 1 1 5E0A347E
 P 6900 4100
-F 0 "C1" H 6992 4146 50  0000 L CNN
+F 0 "C16" H 6992 4146 50  0000 L CNN
 F 1 "2.2u" H 6992 4055 50  0000 L CNN
 F 2 "Capacitor_SMD:C_0603_1608Metric" H 6900 4100 50  0001 C CNN
@@
 $EndComp
 $Comp
-L Device:C_Small C4
+L Device:C_Small C22
 U 1 1 5E0A4446
 P 9900 4550
-F 0 "C4" H 9992 4596 50  0000 L CNN
+F 0 "C22" H 9992 4596 50  0000 L CNN
 F 1 "2.2u" H 9992 4505 50  0000 L CNN
 F 2 "Capacitor_SMD:C_0603_1608Metric" H 9900 4550 50  0001 C CNN
@@
 $EndComp
 $Comp
-L Device:C_Small C5
+L Device:C_Small C23
 U 1 1 5E0A48A0
 P 9900 4950
-F 0 "C5" H 9992 4996 50  0000 L CNN
+F 0 "C23" H 9992 4996 50  0000 L CNN
 F 1 "2.2u" H 9992 4905 50  0000 L CNN
 F 2 "Capacitor_SMD:C_0603_1608Metric" H 9900 4950 50  0001 C CNN
@@
 $EndComp
 $Comp
-L Device:C_Small C3
+L Device:C_Small C21
 U 1 1 5E0A4B9B
 P 9900 4150
-F 0 "C3" H 9808 4196 50  0000 R CNN
+F 0 "C21" H 9808 4196 50  0000 R CNN
 F 1 "4.7u" H 9808 4105 50  0000 R CNN
 F 2 "Capacitor_SMD:C_0603_1608Metric" H 9900 4150 50  0001 C CNN
@@
 $EndComp
 $Comp
-L Device:C_Small C2
+L Device:C_Small C17
 U 1 1 5E0A50B8
 P 6950 4850
-F 0 "C2" H 7042 4896 50  0000 L CNN
+F 0 "C17" H 7042 4896 50  0000 L CNN
 F 1 "1u" H 7042 4805 50  0000 L CNN
 F 2 "Capacitor_SMD:C_0603_1608Metric" H 6950 4850 50  0001 C CNN
@@
 $EndComp
 $Comp
-L favorites:MCP16311_2 U13
+L favorites:MCP16311_2 U3
 U 1 1 5E0A8AEC
 P 7500 1950
-F 0 "U13" H 7500 2250 60  0000 C CNN
+F 0 "U3" H 7500 2250 60  0000 C CNN
 F 1 "MCP16311_2" H 7500 1650 60  0000 C CNN
 F 2 "" H 7550 1950 60  0001 C CNN

Commit message: tweaks
Parts:
- U3: footprint (none) -> Package_SO:MSOP-8_3x3mm_P0.65mm; OrderN (none) -> MCP16311T-E/MSCT-ND
Other:
- note added: "Connected at power source\n"
Changed lines of the file:
@@
 $Descr A4 11693 8268
 encoding utf-8
-Sheet 3 4
-Title ""
+Sheet 2 4
+Title "SYNTH"
 Date ""
-Rev ""
-Comp ""
+Rev "1"
+Comp "Bo Joel Svensson"
 Comment1 ""
 Comment2 ""
@@
 F 0 "U3" H 7500 2250 60  0000 C CNN
 F 1 "MCP16311_2" H 7500 1650 60  0000 C CNN
-F 2 "" H 7550 1950 60  0001 C CNN
+F 2 "Package_SO:MSOP-8_3x3mm_P0.65mm" H 7550 1950 60  0001 C CNN
 F 3 "" H 7550 1950 60  0000 C CNN
+F 4 "MCP16311T-E/MSCT-ND" H 7500 1950 50  0001 C CNN "OrderN"
 	1    7500 1950
 	1    0    0    -1
 $EndComp
+Text Notes 1850 2250 0    50   ~ 0
+Connected at power source\n
+$Comp
+L power:GNDA #PWR016
+U 1 1 5E0B651C
+P 2600 1900
+F 0 "#PWR016" H 2600 1650 50  0001 C CNN
+F 1 "GNDA" H 2605 1727 50  0000 C CNN
+F 2 "" H 2600 1900 50  0001 C CNN
+F 3 "" H 2600 1900 50  0001 C CNN
+	1    2600 1900
+	1    0    0    -1
+$EndComp
+$Comp
+L power:GND #PWR015
+U 1 1 5E0B620C
+P 2100 1900
+F 0 "#PWR015" H 2100 1650 50  0001 C CNN
+F 1 "GND" H 2105 1727 50  0000 C CNN
+F 2 "" H 2100 1900 50  0001 C CNN
+F 3 "" H 2100 1900 50  0001 C CNN
+	1    2100 1900
+	1    0    0    -1
+$EndComp
+$Comp
+L power:PWR_FLAG #FLG01
+U 1 1 5E0B7648
+P 2100 1750
+F 0 "#FLG01" H 2100 1825 50  0001 C CNN
+F 1 "PWR_FLAG" H 2100 1923 50  0000 C CNN
+F 2 "" H 2100 1750 50  0001 C CNN
+F 3 "~" H 2100 1750 50  0001 C CNN
+	1    2100 1750
+	1    0    0    -1
+$EndComp
+$Comp
+L power:PWR_FLAG #FLG02
+U 1 1 5E0B7923
+P 2600 1750
+F 0 "#FLG02" H 2600 1825 50  0001 C CNN
+F 1 "PWR_FLAG" H 2600 1923 50  0000 C CNN
+F 2 "" H 2600 1750 50  0001 C CNN
+F 3 "~" H 2600 1750 50  0001 C CNN
+	1    2600 1750
+	1    0    0    -1
+$EndComp
+Wire Wire Line
+	2100 1900 2100 1750
+Wire Wire Line
+	2600 1900 2600 1750
+$Comp
+L power:+5V #PWR0101
+U 1 1 5E0E43A9
+P 3600 1700
+F 0 "#PWR0101" H 3600 1550 50  0001 C CNN
+F 1 "+5V" H 3615 1873 50  0000 C CNN
+F 2 "" H 3600 1700 50  0001 C CNN
+F 3 "" H 3600 1700 50  0001 C CNN
+	1    3600 1700
+	1    0    0    -1
+$EndComp
+$Comp
+L power:PWR_FLAG #FLG0101
+U 1 1 5E0E4EC0
+P 3600 1950
+F 0 "#FLG0101" H 3600 2025 50  0001 C CNN
+F 1 "PWR_FLAG" H 3600 2123 50  0000 C CNN
+F 2 "" H 3600 1950 50  0001 C CNN
+F 3 "~" H 3600 1950 50  0001 C CNN
+	1    3600 1950
+	-1   0    0    1
+$EndComp
+Wire Wire Line
+	3600 1950 3600 1700
 $EndSCHEMATC

Commit message: low energy work
Parts:
- added R10: 91k, Resistor_SMD:R_0603_1608Metric, symbol Device:R_Small
- added R9: 249k, Resistor_SMD:R_0603_1608Metric, symbol Device:R_Small
- added U2: REF3030, Package_TO_SOT_SMD:SOT-23, symbol Reference_Voltage:REF3030
- renumbered C19 to C10, C20 to C11, C16 to C2, C17 to C3, C21 to C4, C14 to C5, C22 to C6, C23 to C7, C15 to C8, C18 to C9, R12 to R11, R14 to R12, R11 to R13, R13 to R14, R10 to R8, U2 to U1
Connections:
- net +3V3: now also U2.1 (IN)
- net +5V: now also C2.1, R8.1, U1.12 (EN+), U1.3 (VIN), U1.8 (EN-)
- net GND: now also C2.2, C4.2, C6.2, C7.2, R12.2, U1.13 (PAD), U1.4 (GND), R10.2, U2.3 (GND)
- net at U1.1 (PGOOD): now also R8.2
- net at U1.10 (C+): now also C3.1
- net RAIL+: now reaches U1.11 (OUT+)
- net RAIL+: now also C6.1, R11.1
- net at U1.2 (FB+): now also R11.2, R12.1
- net at U1.5 (CP): now also C4.1
- net RAIL-: now reaches U1.6 (OUT-)
- net RAIL-: now also C7.1, R10.1, R9.2
- net at U1.7 (FB-): now also R9.1
- net at U1.9 (C-): now also C3.2
- new net VREF: U2.2 (OUT)
Other:
- moved on the sheet: C2, C3, C4, C6, C7, R11, R12, R8

Commit message: update
Other:
- note removed: "Connected at power source\n"
Changed lines of the file:
@@
 	6750 1250 6750 1450
 Wire Wire Line
-	9250 1250 9250 1700
+	9250 1250 9250 1600
 Wire Wire Line
 	8300 1900 8300 1550
@@
 $EndComp
 $Comp
-L power:GND #PWR014
+L power:GND #PWR013
 U 1 1 5B1BFD77
 P 8200 2700
-F 0 "#PWR014" H 8200 2450 50  0001 C CNN
+F 0 "#PWR013" H 8200 2450 50  0001 C CNN
 F 1 "GND" H 8200 2550 50  0000 C CNN
 F 2 "" H 8200 2700 60  0000 C CNN
@@
 	6750 2450 6750 2600
 $Comp
-L power:+5V #PWR012
+L power:+5V #PWR011
 U 1 1 5DD19B4C
 P 6500 1700
-F 0 "#PWR012" H 6500 1550 50  0001 C CNN
+F 0 "#PWR011" H 6500 1550 50  0001 C CNN
 F 1 "+5V" H 6515 1873 50  0000 C CNN
 F 2 "" H 6500 1700 50  0001 C CNN
@@
 $EndComp
 $Comp
-L power:+3V3 #PWR015
+L power:+3V3 #PWR014
 U 1 1 5E0CE9A5
 P 9050 1650
-F 0 "#PWR015" H 9050 1500 50  0001 C CNN
+F 0 "#PWR014" H 9050 1500 50  0001 C CNN
 F 1 "+3V3" H 9065 1823 50  0000 C CNN
 F 2 "" H 9050 1650 50  0001 C CNN
@@
 	1    0    0    -1
 $EndComp
-Text Notes 1850 2250 0    50   ~ 0
-Connected at power source\n
-$Comp
-L power:GNDA #PWR04
-U 1 1 5E0B651C
-P 2600 1900
-F 0 "#PWR04" H 2600 1650 50  0001 C CNN
-F 1 "GNDA" H 2605 1727 50  0000 C CNN
-F 2 "" H 2600 1900 50  0001 C CNN
-F 3 "" H 2600 1900 50  0001 C CNN
-	1    2600 1900
-	1    0    0    -1
-$EndComp
 $Comp
 L power:GND #PWR03
@@
 	1    0    0    -1
 $EndComp
-$Comp
-L power:PWR_FLAG #FLG02
-U 1 1 5E0B7923
-P 2600 1750
-F 0 "#FLG02" H 2600 1825 50  0001 C CNN
-F 1 "PWR_FLAG" H 2600 1923 50  0000 C CNN
-F 2 "" H 2600 1750 50  0001 C CNN
-F 3 "~" H 2600 1750 50  0001 C CNN
-	1    2600 1750
-	1    0    0    -1
-$EndComp
 Wire Wire Line
 	2100 1900 2100 1750
-Wire Wire Line
-	2600 1900 2600 1750
-$Comp
-L power:+5V #PWR05
+$Comp
+L power:+5V #PWR04
 U 1 1 5E0E43A9
 P 3600 1700
-F 0 "#PWR05" H 3600 1550 50  0001 C CNN
+F 0 "#PWR04" H 3600 1550 50  0001 C CNN
 F 1 "+5V" H 3615 1873 50  0000 C CNN
 F 2 "" H 3600 1700 50  0001 C CNN
@@
 $EndComp
 $Comp
-L power:PWR_FLAG #FLG03
+L power:PWR_FLAG #FLG02
 U 1 1 5E0E4EC0
 P 3600 1950
-F 0 "#FLG03" H 3600 2025 50  0001 C CNN
+F 0 "#FLG02" H 3600 2025 50  0001 C CNN
 F 1 "PWR_FLAG" H 3600 2123 50  0000 C CNN
 F 2 "" H 3600 1950 50  0001 C CNN
@@
 $EndComp
 $Comp
-L power:+3V3 #PWR08
+L power:+3V3 #PWR07
 U 1 1 5E0AC242
 P 5100 2700
-F 0 "#PWR08" H 5100 2550 50  0001 C CNN
+F 0 "#PWR07" H 5100 2550 50  0001 C CNN
 F 1 "+3V3" H 5115 2873 50  0000 C CNN
 F 2 "" H 5100 2700 50  0001 C CNN
@@
 	5500 3100 5800 3100
 $Comp
-L power:GND #PWR09
+L power:GND #PWR08
 U 1 1 5E0ACBE4
 P 5100 3600
-F 0 "#PWR09" H 5100 3350 50  0001 C CNN
+F 0 "#PWR08" H 5100 3350 50  0001 C CNN
 F 1 "GND" H 5105 3427 50  0000 C CNN
 F 2 "" H 5100 3600 50  0001 C CNN
@@
 	5100 3600 5100 3400
 $Comp
-L power:+5V #PWR06
+L power:+5V #PWR05
 U 1 1 5E0AE864
 P 3750 4150
-F 0 "#PWR06" H 3750 4000 50  0001 C CNN
+F 0 "#PWR05" H 3750 4000 50  0001 C CNN
 F 1 "+5V" H 3765 4323 50  0000 C CNN
 F 2 "" H 3750 4150 50  0001 C CNN
@@
 Connection ~ 3750 4350
 $Comp
-L power:GND #PWR07
+L power:GND #PWR06
 U 1 1 5E0AF975
 P 3750 4700
-F 0 "#PWR07" H 3750 4450 50  0001 C CNN
+F 0 "#PWR06" H 3750 4450 50  0001 C CNN
 F 1 "GND" H 3755 4527 50  0000 C CNN
 F 2 "" H 3750 4700 50  0001 C CNN
@@
 	4300 5200 4300 5150
 $Comp
-L power:GND #PWR010
+L power:GND #PWR09
 U 1 1 5E0B3910
 P 5100 5500
-F 0 "#PWR010" H 5100 5250 50  0001 C CNN
+F 0 "#PWR09" H 5100 5250 50  0001 C CNN
 F 1 "GND" H 5105 5327 50  0000 C CNN
 F 2 "" H 5100 5500 50  0001 C CNN
@@
 	5950 4950 5950 4900
 $Comp
-L power:GND #PWR011
+L power:GND #PWR010
 U 1 1 5E0BA4A0
 P 6300 5350
-F 0 "#PWR011" H 6300 5100 50  0001 C CNN
+F 0 "#PWR010" H 6300 5100 50  0001 C CNN
 F 1 "GND" H 6305 5177 50  0000 C CNN
 F 2 "" H 6300 5350 50  0001 C CNN
@@
 	6300 5300 6300 5350
 $Comp
-L power:GND #PWR013
+L power:GND #PWR012
 U 1 1 5E0BDA29
 P 6700 4650
-F 0 "#PWR013" H 6700 4400 50  0001 C CNN
+F 0 "#PWR012" H 6700 4400 50  0001 C CNN
 F 1 "GND" H 6705 4477 50  0000 C CNN
 F 2 "" H 6700 4650 50  0001 C CNN
@@
 	4450 4750 4450 4650
 Connection ~ 4450 4650
+$Comp
+L power:PWR_FLAG #FLG0101
+U 1 1 5E15F7E2
+P 9250 1600
+F 0 "#FLG0101" H 9250 1675 50  0001 C CNN
+F 1 "PWR_FLAG" V 9250 1728 50  0000 L CNN
+F 2 "" H 9250 1600 50  0001 C CNN
+F 3 "~" H 9250 1600 50  0001 C CNN
+	1    9250 1600
+	0    1    1    0
+$EndComp
+Connection ~ 9250 1600
+Wire Wire Line
+	9250 1600 9250 1700
 $EndSCHEMATC

Commit message: experimenting
Parts:
- added C29: 100u, Capacitor_THT:CP_Radial_D10.0mm_P5.00mm, symbol Device:CP_Small
- added C30: 2.2u, Capacitor_SMD:C_0603_1608Metric, symbol Device:C_Small
- U1: OrderN (none) -> 296-47331-1-ND
Connections:
- net +3V3: now also C30.2
- net +5V: now also C29.1
- net GND: now also C29.2, C30.1
Other:
- note added: "Close to USB port\n"
Changed lines of the file:
@@
 F 2 "Package_SON:WSON-12-1EP_3x2mm_P0.5mm_EP1x2.65_ThermalVias" H 5200 3800 50  0001 L CNN
 F 3 "http://www.ti.com/lit/ds/symlink/lm27762.pdf" H 7550 4150 50  0001 C CNN
+F 4 " 296-47331-1-ND " H 5050 4550 50  0001 C CNN "OrderN"
 	1    5050 4550
 	1    0    0    -1
@@
 $EndComp
 Wire Wire Line
-	5100 2800 5100 2700
+	5100 2800 5100 2750
 Text HLabel 5800 3100 2    50   Input ~ 0
 VREF
@@
 Wire Wire Line
 	9250 1600 9250 1700
+$Comp
+L Device:CP_Small C29
+U 1 1 5E13C1F9
+P 4550 1900
+F 0 "C29" V 4774 1900 50  0000 C CNN
+F 1 "100u" V 4683 1900 50  0000 C CNN
+F 2 "Capacitor_THT:CP_Radial_D10.0mm_P5.00mm" H 4550 1900 50  0001 C CNN
+F 3 "~" H 4550 1900 50  0001 C CNN
+F 4 "493-11829-1-ND " V 4550 1900 50  0001 C CNN "OrderN"
+	1    4550 1900
+	0    -1   -1   0
+$EndComp
+$Comp
+L power:+5V #PWR0102
+U 1 1 5E13EC1A
+P 4300 1700
+F 0 "#PWR0102" H 4300 1550 50  0001 C CNN
+F 1 "+5V" H 4315 1873 50  0000 C CNN
+F 2 "" H 4300 1700 50  0001 C CNN
+F 3 "" H 4300 1700 50  0001 C CNN
+	1    4300 1700
+	1    0    0    -1
+$EndComp
+$Comp
+L power:GND #PWR0103
+U 1 1 5E13F0A2
+P 4850 2050
+F 0 "#PWR0103" H 4850 1800 50  0001 C CNN
+F 1 "GND" H 4855 1877 50  0000 C CNN
+F 2 "" H 4850 2050 50  0001 C CNN
+F 3 "" H 4850 2050 50  0001 C CNN
+	1    4850 2050
+	1    0    0    -1
+$EndComp
+Wire Wire Line
+	4850 2050 4850 1900
+Wire Wire Line
+	4650 1900 4850 1900
+Wire Wire Line
+	4450 1900 4300 1900
+Wire Wire Line
+	4300 1900 4300 1700
+Text Notes 4750 1750 0    50   ~ 0
+Close to USB port\n
+$Comp
+L Device:C_Small C30
+U 1 1 5E15487E
+P 5400 2750
+F 0 "C30" H 5425 2850 50  0000 L CNN
+F 1 "2.2u" V 5250 2700 50  0000 L CNN
+F 2 "Capacitor_SMD:C_0603_1608Metric" H 5438 2600 30  0001 C CNN
+F 3 "" H 5400 2750 60  0000 C CNN
+F 4 " 490-10731-1-ND " H 5400 2750 50  0001 C CNN "OrderN"
+	1    5400 2750
+	0    1    1    0
+$EndComp
+$Comp
+L power:GND #PWR021
+U 1 1 5E155C89
+P 5650 2800
+F 0 "#PWR021" H 5650 2550 50  0001 C CNN
+F 1 "GND" H 5655 2627 50  0000 C CNN
+F 2 "" H 5650 2800 50  0001 C CNN
+F 3 "" H 5650 2800 50  0001 C CNN
+	1    5650 2800
+	1    0    0    -1
+$EndComp
+Wire Wire Line
+	5650 2800 5650 2750
+Wire Wire Line
+	5650 2750 5500 2750
+Wire Wire Line
+	5100 2750 5300 2750
+Connection ~ 5100 2750
+Wire Wire Line
+	5100 2750 5100 2700
 $EndSCHEMATC

Commit message: I found a bug
Parts:
- C10, C30, C5, C8: OrderN 490-10731-1-ND -> 490-10731-1-ND
- C11: OrderN 478-5651-1-ND -> 478-5651-1-ND
- C2, C6, C7: OrderN (none) -> 490-10731-1-ND
- C3: OrderN (none) -> 1276-6524-1-ND
- C4: OrderN (none) -> 587-1441-1-ND
- R10, R12: OrderN (none) -> 311-91.0KHRCT-ND
- R11, R9: OrderN (none) -> 311-249KHRCT-ND
- R14: OrderN 311-10.0KHRDKR-ND -> 311-10.0KHRCT-ND
- R8: OrderN (none) -> 311-10.0KHRCT-ND
Changed lines of the file:
@@
 F 2 "Capacitor_SMD:C_0603_1608Metric" H 6538 2200 30  0001 C CNN
 F 3 "" H 6500 2350 60  0000 C CNN
-F 4 " 490-10731-1-ND " H 6500 2350 50  0001 C CNN "OrderN"
+F 4 "490-10731-1-ND" H 6500 2350 50  0001 C CNN "OrderN"
 	1    6500 2350
 	1    0    0    -1
@@
 F 2 "Capacitor_SMD:C_0603_1608Metric" H 6788 2200 30  0001 C CNN
 F 3 "" H 6750 2350 60  0000 C CNN
-F 4 " 490-10731-1-ND " H 6750 2350 50  0001 C CNN "OrderN"
+F 4 "490-10731-1-ND" H 6750 2350 50  0001 C CNN "OrderN"
 	1    6750 2350
 	1    0    0    -1
@@
 F 2 "Capacitor_SMD:C_0603_1608Metric" H 9038 2200 30  0001 C CNN
 F 3 "" H 9000 2350 60  0000 C CNN
-F 4 " 490-10731-1-ND " H 9000 2350 50  0001 C CNN "OrderN"
+F 4 "490-10731-1-ND" H 9000 2350 50  0001 C CNN "OrderN"
 	1    9000 2350
 	1    0    0    -1
@@
 F 2 "Capacitor_Tantalum_SMD:CP_EIA-3528-12_Kemet-T" H 9250 2350 60  0001 C CNN
 F 3 "" H 9250 2350 60  0000 C CNN
-F 4 " 478-5651-1-ND" H 9250 2350 50  0001 C CNN "OrderN"
+F 4 "478-5651-1-ND" H 9250 2350 50  0001 C CNN "OrderN"
 	1    9250 2350
 	1    0    0    -1
@@
 F 2 "Resistor_SMD:R_0603_1608Metric" V 7730 1450 30  0001 C CNN
 F 3 "" H 7800 1450 30  0000 C CNN
-F 4 "311-10.0KHRDKR-ND " H 7800 1450 50  0001 C CNN "OrderN"
+F 4 " 311-10.0KHRCT-ND" H 7800 1450 50  0001 C CNN "OrderN"
 	1    7800 1450
 	0    1    1    0
@@
 F 2 "Resistor_SMD:R_0603_1608Metric" H 6300 4400 50  0001 C CNN
 F 3 "~" H 6300 4400 50  0001 C CNN
+F 4 "311-249KHRCT-ND " H 6300 4400 50  0001 C CNN "OrderN"
 	1    6300 4400
 	1    0    0    -1
@@
 F 2 "Resistor_SMD:R_0603_1608Metric" H 6300 4700 50  0001 C CNN
 F 3 "~" H 6300 4700 50  0001 C CNN
+F 4 " 311-91.0KHRCT-ND" H 6300 4700 50  0001 C CNN "OrderN"
 	1    6300 4700
 	1    0    0    -1
@@
 F 2 "Resistor_SMD:R_0603_1608Metric" H 4050 4450 50  0001 C CNN
 F 3 "~" H 4050 4450 50  0001 C CNN
+F 4 " 311-10.0KHRCT-ND" H 4050 4450 50  0001 C CNN "OrderN"
 	1    4050 4450
 	1    0    0    -1
@@
 F 2 "Capacitor_SMD:C_0603_1608Metric" H 3750 4450 50  0001 C CNN
 F 3 "~" H 3750 4450 50  0001 C CNN
+F 4 "490-10731-1-ND" H 3750 4450 50  0001 C CNN "OrderN"
 	1    3750 4450
 	1    0    0    -1
@@
 F 2 "Capacitor_SMD:C_0603_1608Metric" H 6700 4400 50  0001 C CNN
 F 3 "~" H 6700 4400 50  0001 C CNN
+F 4 "490-10731-1-ND" H 6700 4400 50  0001 C CNN "OrderN"
 	1    6700 4400
 	1    0    0    -1
@@
 F 2 "Capacitor_SMD:C_0603_1608Metric" H 6700 5150 50  0001 C CNN
 F 3 "~" H 6700 5150 50  0001 C CNN
+F 4 "490-10731-1-ND" H 6700 5150 50  0001 C CNN "OrderN"
 	1    6700 5150
 	1    0    0    -1
@@
 F 2 "Capacitor_SMD:C_0603_1608Metric" H 5650 5350 50  0001 C CNN
 F 3 "~" H 5650 5350 50  0001 C CNN
+F 4 " 587-1441-1-ND " H 5650 5350 50  0001 C CNN "OrderN"
 	1    5650 5350
 	1    0    0    -1
@@
 F 2 "Capacitor_SMD:C_0603_1608Metric" H 4300 5050 50  0001 C CNN
 F 3 "~" H 4300 5050 50  0001 C CNN
+F 4 "1276-6524-1-ND " H 4300 5050 50  0001 C CNN "OrderN"
 	1    4300 5050
 	1    0    0    -1
@@
 F 2 "Resistor_SMD:R_0603_1608Metric" H 5950 4800 50  0001 C CNN
 F 3 "~" H 5950 4800 50  0001 C CNN
+F 4 "311-249KHRCT-ND " H 5950 4800 50  0001 C CNN "OrderN"
 	1    5950 4800
 	1    0    0    -1
@@
 F 2 "Resistor_SMD:R_0603_1608Metric" H 5950 5100 50  0001 C CNN
 F 3 "~" H 5950 5100 50  0001 C CNN
+F 4 " 311-91.0KHRCT-ND" H 5950 5100 50  0001 C CNN "OrderN"
 	1    5950 5100
 	1    0    0    -1
@@
 F 2 "Capacitor_SMD:C_0603_1608Metric" H 5438 2600 30  0001 C CNN
 F 3 "" H 5400 2750 60  0000 C CNN
-F 4 " 490-10731-1-ND " H 5400 2750 50  0001 C CNN "OrderN"
+F 4 "490-10731-1-ND" H 5400 2750 50  0001 C CNN "OrderN"
 	1    5400 2750
 	0    1    1    0
