File: Hardware/V1_0/Information.sch (KiCad schematic (older format))
At the start: 11 parts, among them J1 AudioJack3_Ground, U10 AD5330, U11 CAT5113, U12 CAT5113, U2 AD5341, U3 AD5341, U4 LF356, U5 LF356, U6 OP295, U8 AD5330, U9 SN74HC139

Commit message: some work on the MCU part
Parts:
- removed J1: AudioJack3_Ground, symbol Connector:AudioJack3_Ground
- removed U6: OP295, symbol favorites:OP295
- added J?ee1: AudioJack3_Ground, v2_0:Jack_3.5mm_CUI_SJ-3524-SMT_Horizontal, symbol Connector:AudioJack3_Ground
- added U9: REF3030, Package_TO_SOT_SMD:SOT-23, symbol Reference_Voltage:REF3030
- renumbered U4 to U10, U5 to U11, U11 to U12, U12 to U13, U8 to U4, U9 to U5, U10 to U6, U2 to U7, U3 to U8
Connections:
- wire segments 11 -> 5
- no-connect marks 0 -> 2
Changed lines of the file:
@@
 $EndDescr
 $Comp
-L favorites:AD5341 U2
+L favorites:AD5341 U7
 U 1 1 5E06F395
 P 4150 2950
-F 0 "U2" H 4150 2135 50  0000 C CNN
+F 0 "U7" H 4150 2135 50  0000 C CNN
 F 1 "AD5341" H 4150 2226 50  0000 C CNN
 F 2 "Package_SO:TSSOP-20_4.4x6.5mm_P0.65mm" H 4000 2950 50  0001 C CNN
@@
 Text Notes 4500 3700 0    50   ~ 0
 \nAD5341BRUZ-REEL7
-$Comp
-L favorites:OP295 U6
-U 1 1 5E0717D4
-P 6600 3350
-F 0 "U6" H 6600 3865 50  0000 C CNN
-F 1 "OP295" H 6600 3774 50  0000 C CNN
-F 2 "" H 6600 3350 50  0001 C CNN
-F 3 "" H 6600 3350 50  0001 C CNN
-	1    6600 3350
-	1    0    0    -1
-$EndComp
-$Comp
-L power:GND #PWR0101
-U 1 1 5E075500
-P 6600 3800
-F 0 "#PWR0101" H 6600 3550 50  0001 C CNN
-F 1 "GND" H 6605 3627 50  0000 C CNN
-F 2 "" H 6600 3800 50  0001 C CNN
-F 3 "" H 6600 3800 50  0001 C CNN
-	1    6600 3800
-	1    0    0    -1
-$EndComp
-Wire Wire Line
-	7000 3450 7200 3450
-Wire Wire Line
-	7200 3450 7200 3800
-Wire Wire Line
-	7200 3800 6600 3800
-Wire Wire Line
-	6600 3800 5900 3800
-Wire Wire Line
-	5900 3800 5900 3350
-Wire Wire Line
-	5900 3350 6200 3350
-Connection ~ 6600 3800
-$Comp
-L Connector:AudioJack3_Ground J1
-U 1 1 5E075F59
-P 6750 1850
-F 0 "J1" H 6732 2175 50  0000 C CNN
-F 1 "AudioJack3_Ground" H 6732 2084 50  0000 C CNN
-F 2 "" H 6750 1850 50  0001 C CNN
-F 3 "~" H 6750 1850 50  0001 C CNN
-	1    6750 1850
-	1    0    0    -1
-$EndComp
 $Bitmap
 Pos 10400 1000
@@
 Line level\n
 $Comp
-L power:GND #PWR0102
+L power:GND #PWR025
 U 1 1 5E06DF17
 P 6750 2350
-F 0 "#PWR0102" H 6750 2100 50  0001 C CNN
+F 0 "#PWR025" H 6750 2100 50  0001 C CNN
 F 1 "GND" H 6755 2177 50  0000 C CNN
 F 2 "" H 6750 2350 50  0001 C CNN
@@
 	6750 2250 6750 2150
 $Comp
-L Amplifier_Operational:LF356 U4
+L Amplifier_Operational:LF356 U10
 U 1 1 5E0760F9
 P 6550 4550
-F 0 "U4" H 6894 4596 50  0000 L CNN
+F 0 "U10" H 6894 4596 50  0000 L CNN
 F 1 "LF356" H 6894 4505 50  0000 L CNN
 F 2 "Package_SO:SOIC-8_3.9x4.9mm_P1.27mm" H 6600 4600 50  0001 C CNN
@@
 $EndComp
 $Comp
-L Amplifier_Operational:LF356 U5
+L Amplifier_Operational:LF356 U11
 U 1 1 5E07878A
 P 6550 5350
-F 0 "U5" H 6894 5396 50  0000 L CNN
+F 0 "U11" H 6894 5396 50  0000 L CNN
 F 1 "LF356" H 6894 5305 50  0000 L CNN
 F 2 "Package_SO:SOIC-8_3.9x4.9mm_P1.27mm" H 6600 5400 50  0001 C CNN
@@
 $EndComp
 $Comp
-L favorites:AD5341 U3
+L favorites:AD5341 U8
 U 1 1 5E07AF77
 P 4150 4500
-F 0 "U3" H 4150 3685 50  0000 C CNN
+F 0 "U8" H 4150 3685 50  0000 C CNN
 F 1 "AD5341" H 4150 3776 50  0000 C CNN
 F 2 "Package_SO:TSSOP-20_4.4x6.5mm_P0.65mm" H 4000 4500 50  0001 C CNN
@@
 http://dangerousprototypes.com/blog/2010/03/29/play-wav-audio-files-with-ad5330-and-arduino/
 $Comp
-L favorites:CAT5113 U11
+L favorites:CAT5113 U12
 U 1 1 5E080859
 P 8500 3650
-F 0 "U11" H 8475 4115 50  0000 C CNN
+F 0 "U12" H 8475 4115 50  0000 C CNN
 F 1 "CAT5113" H 8475 4024 50  0000 C CNN
 F 2 "Package_SO:SOIC-8-N7_3.9x4.9mm_P1.27mm" H 8500 3200 50  0001 C CNN
@@
 $EndComp
 $Comp
-L favorites:CAT5113 U12
+L favorites:CAT5113 U13
 U 1 1 5E080A1E
 P 8500 4800
-F 0 "U12" H 8475 5265 50  0000 C CNN
+F 0 "U13" H 8475 5265 50  0000 C CNN
 F 1 "CAT5113" H 8475 5174 50  0000 C CNN
 F 2 "Package_SO:SOIC-8-N7_3.9x4.9mm_P1.27mm" H 8500 4350 50  0001 C CNN
@@
 $EndComp
 $Comp
-L favorites:SN74HC139 U9
+L favorites:SN74HC139 U5
 U 1 1 5E0896B0
 P 2000 2950
-F 0 "U9" H 2000 3565 50  0000 C CNN
+F 0 "U5" H 2000 3565 50  0000 C CNN
 F 1 "SN74HC139" H 2000 3474 50  0000 C CNN
 F 2 "" H 1900 2850 50  0001 C CNN
@@
 $EndComp
 $Comp
-L favorites:AD5330 U8
+L favorites:AD5330 U4
 U 1 1 5E08A77E
 P 1650 6550
-F 0 "U8" H 1650 7315 50  0000 C CNN
+F 0 "U4" H 1650 7315 50  0000 C CNN
 F 1 "AD5330" H 1650 7224 50  0000 C CNN
 F 2 "Package_SO:TSSOP-20_4.4x6.5mm_P0.65mm" H 1650 6550 50  0001 C CNN
@@
 $EndComp
 $Comp
-L favorites:AD5330 U10
+L favorites:AD5330 U6
 U 1 1 5E08C0E0
 P 3200 6550
-F 0 "U10" H 3200 7315 50  0000 C CNN
+F 0 "U6" H 3200 7315 50  0000 C CNN
 F 1 "AD5330" H 3200 7224 50  0000 C CNN
 F 2 "" H 3200 6550 50  0001 C CNN
@@
 	1    0    0    -1
 $EndComp
+$Comp
+L Reference_Voltage:REF3030 U9
+U 1 1 5E0A14BA
+P 4350 5500
+F 0 "U9" H 4121 5546 50  0000 R CNN
+F 1 "REF3030" H 4121 5455 50  0000 R CIN
+F 2 "Package_TO_SOT_SMD:SOT-23" H 4350 5050 50  0001 C CIN
+F 3 "http://www.ti.com/lit/ds/symlink/ref3033.pdf" H 4450 5150 50  0001 C CIN
+F 4 " 296-26323-2-ND " H 4350 5500 50  0001 C CNN "OrderN"
+	1    4350 5500
+	1    0    0    -1
+$EndComp
+$Comp
+L Connector:AudioJack3_Ground J?ee1
+U 1 1 5DD862BF
+P 6750 1850
+F 0 "J?ee1" H 6732 2175 50  0000 C CNN
+F 1 "AudioJack3_Ground" H 6732 2084 50  0000 C CNN
+F 2 "v2_0:Jack_3.5mm_CUI_SJ-3524-SMT_Horizontal" H 6750 1850 50  0001 C CNN
+F 3 "~" H 6750 1850 50  0001 C CNN
+F 4 "CP-3524SJCT-ND " H 6750 1850 50  0001 C CNN "OrderN"
+	1    6750 1850
+	1    0    0    -1
+$EndComp
+NoConn ~ 6950 1850
+NoConn ~ 6950 1950
 $EndSCHEMATC

Commit message: tweaks
Parts:
- U12, U13: OrderN (none) -> CAT5113VI-01-GT3OSCT-ND
- U4: OrderN (none) -> AD5330BRUZ-ND
- U5: footprint (none) -> Package_SO:SOIC-16_3.9x9.9mm_P1.27mm; OrderN (none) -> 296-14833-2-ND
- U6: footprint (none) -> Package_SO:TSSOP-20_4.4x6.5mm_P0.65mm; OrderN (none) -> AD5330BRUZ-ND
Changed lines of the file:
@@
 $Descr A4 11693 8268
 encoding utf-8
-Sheet 4 4
-Title ""
+Sheet 3 4
+Title "SYNTH"
 Date ""
-Rev ""
-Comp ""
+Rev "1"
+Comp "Bo Joel Svensson"
 Comment1 ""
 Comment2 ""
@@
 F 2 "Package_SO:SOIC-8-N7_3.9x4.9mm_P1.27mm" H 8500 3200 50  0001 C CNN
 F 3 "" H 8400 3450 50  0001 C CNN
+F 4 " CAT5113VI-01-GT3OSCT-ND " H 8500 3650 50  0001 C CNN "OrderN"
 	1    8500 3650
 	1    0    0    -1
@@
 F 2 "Package_SO:SOIC-8-N7_3.9x4.9mm_P1.27mm" H 8500 4350 50  0001 C CNN
 F 3 "" H 8400 4600 50  0001 C CNN
+F 4 " CAT5113VI-01-GT3OSCT-ND " H 8500 4800 50  0001 C CNN "OrderN"
 	1    8500 4800
 	1    0    0    -1
@@
 F 0 "U5" H 2000 3565 50  0000 C CNN
 F 1 "SN74HC139" H 2000 3474 50  0000 C CNN
-F 2 "" H 1900 2850 50  0001 C CNN
+F 2 "Package_SO:SOIC-16_3.9x9.9mm_P1.27mm" H 1900 2850 50  0001 C CNN
 F 3 "" H 1900 2850 50  0001 C CNN
+F 4 " 296-14833-2-ND " H 2000 2950 50  0001 C CNN "OrderN"
 	1    2000 2950
 	1    0    0    -1
@@
 F 2 "Package_SO:TSSOP-20_4.4x6.5mm_P0.65mm" H 1650 6550 50  0001 C CNN
 F 3 "" H 1650 6550 50  0001 C CNN
+F 4 "AD5330BRUZ-ND" H 1650 6550 50  0001 C CNN "OrderN"
 	1    1650 6550
 	1    0    0    -1
@@
 F 0 "U6" H 3200 7315 50  0000 C CNN
 F 1 "AD5330" H 3200 7224 50  0000 C CNN
-F 2 "" H 3200 6550 50  0001 C CNN
+F 2 "Package_SO:TSSOP-20_4.4x6.5mm_P0.65mm" H 3200 6550 50  0001 C CNN
 F 3 "" H 3200 6550 50  0001 C CNN
+F 4 "AD5330BRUZ-ND" H 3200 6550 50  0001 C CNN "OrderN"
 	1    3200 6550
 	1    0    0    -1

Commit message: low energy work
Parts:
- removed U9: REF3030, Package_TO_SOT_SMD:SOT-23, symbol Reference_Voltage:REF3030
- added C24, C25, C26, C27, C28, C29, C30: 2.2u, Capacitor_SMD:C_0603_1608Metric, symbol Device:C_Small
- renumbered U4 to U5, U5 to U6, U6 to U7, U7 to U8, U8 to U9
Connections:
- net GND: now also U6.1 (N_G_1), U6.8 (GND), C24.2, C25.2, C26.2, C27.2, C28.2, C29.2, C30.2
- net CS0: now reaches U8.6 (NCS)
- net CS0: now also U6.4 (OUT_1_0)
- net CS1: now reaches U9.6 (NCS)
- net CS1: now also U6.5 (OUT_1_1)
- net +3V3: now reaches U6.16 (VCC)
- net +3V3: now also C24.1, C25.1, C26.1, C27.1, C28.1, C29.1, C30.1
- net DMUX0: now reaches U6.2 (A_1)
- net DMUX1: now reaches U6.3 (B_1)
- net CS2: now reaches U6.6 (OUT_1_2)
- net CS2: now also U5.6 (N_CS)
- net CS3: now reaches U6.7 (OUT_1_3)
- net CS3: now also U7.6 (N_CS)
- no-connect marks 2 -> 9
Other:
- moved on the sheet: U6

Commit message: update
Parts:
- removed C24, C29, C30: 2.2u, Capacitor_SMD:C_0603_1608Metric, symbol Device:C_Small
- removed U11: LF356, Package_SO:SOIC-8_3.9x4.9mm_P1.27mm, symbol Amplifier_Operational:LF356
- removed U12, U13: CAT5113, Package_SO:SOIC-8-N7_3.9x4.9mm_P1.27mm, symbol favorites:CAT5113
- removed U6: SN74HC139, Package_SO:SOIC-16_3.9x9.9mm_P1.27mm, symbol favorites:SN74HC139
- removed U7: AD5330, Package_SO:TSSOP-20_4.4x6.5mm_P0.65mm, symbol favorites:AD5330
- removed U8, U9: AD5341, Package_SO:TSSOP-20_4.4x6.5mm_P0.65mm, symbol favorites:AD5341
- added C24: 10u, Capacitor_Tantalum_SMD:CP_EIA-3216-18_Kemet-A, symbol Device:CP_Small
- added J10, J5, J6, J7, J8, J9: C, Connector_PinHeader_2.54mm:PinHeader_1x02_P2.54mm_Vertical, symbol Connector:Conn_01x02_Female
- added J11: AUDIO, Connector_JST:JST_PH_B2B-PH-K_1x02_P2.00mm_Vertical, symbol Connector:Conn_01x02_Male
- added R17, R18, R20, R22, R24: 10k, Resistor_SMD:R_0603_1608Metric, symbol Device:R_Small
- added R19, R21, R23: 30k, Resistor_SMD:R_0603_1608Metric, symbol Device:R_Small
- C25: value 2.2u -> 0.1u
- C26, C27, C28: value 2.2u -> 10uF; footprint Capacitor_SMD:C_0603_1608Metric -> Capacitor_SMD:C_0805_2012Metric; OrderN 490-10731-1-ND -> 490-5523-1-ND
- J?ee1: footprint v2_0:Jack_3.5mm_CUI_SJ-3524-SMT_Horizontal -> favorites:Jack_3.5mm_CUI_SJ-3524-SMT_Horizontal
- renumbered U10 to U6
Connections:
- net CS2 is gone; now on net GND: U5.6 (N_CS)
- net +3V3: now also U5.12 (VDD), C24.1, R17.1; no longer C26.1, C27.1, C28.1
- net DAC1: now also C27.2
- net DAC2: now also C28.2
- net DB0: now also U5.13 (DB0)
- net DB1: now also U5.14 (DB1)
- net DB2: now also U5.15 (DB2)
- net DB3: now also U5.16 (DB3)
- net DB4: now also U5.17 (DB4)
- net DB5: now also U5.18 (DB5)
- net DB6: now also U5.19 (DB6)
- net DB7: now also U5.20 (DB7)
- net GND: now also U5.5 (GND), U5.8 (GAIN), U6.3 (+), C24.2, J11.2 (Pin_2); no longer C26.2, C27.2, C28.2
- net RAIL+: now also U6.7 (V+)
- net RAIL-: now also U6.4 (V-)
- net VREF: now also U5.3 (VREF)
- net at J?ee1.R: now also J?ee1.T, U6.6, J11.1 (Pin_1), R24.1
- net at U6.2 (-): now also R18.2, R19.1, R20.2, R21.1, R22.2, R23.1, R24.2
- net BUF_0: now reaches U5.1 (BUF)
- net N_LDAC_0: now reaches U5.10 (N_LDAC)
- net at U5.11 (N_PD): now also R17.2
- net DACOUT: now reaches U5.4 (VOUT)
- net DACOUT: now also C26.2
- net N_WR_0: now reaches U5.7 (N_WR)
- net N_CLR_0: now reaches U5.9 (N_CLR)
- new net: C27.1, J6.1 (Pin_1), J9.1 (Pin_1)
- new net: C28.1, J10.1 (Pin_1), J7.1 (Pin_1)
- new net: J5.2 (Pin_2), R19.2
- new net: J6.2 (Pin_2), R21.2
- new net: J7.2 (Pin_2), R23.2
- new net: J8.2 (Pin_2), R18.1
- new net: J9.2 (Pin_2), R20.1
- new net: J10.2 (Pin_2), R22.1
- new net: C26.1, J5.1 (Pin_1), J8.1 (Pin_1)
- no-connect marks 9 -> 2
Other:
- note removed: "\nAD5341BRUZ-REEL7"
- moved on the sheet: J?ee1, U5, U6

Commit message: experimenting
Changed lines of the file:
@@
 U 1 1 5E0760F9
 P 6050 2550
-F 0 "U6" H 6394 2596 50  0000 L CNN
-F 1 "LF356" H 6394 2505 50  0000 L CNN
+F 0 "U6" H 6150 2800 50  0000 L CNN
+F 1 "LF356" H 6150 2700 50  0000 L CNN
 F 2 "Package_SO:SOIC-8_3.9x4.9mm_P1.27mm" H 6100 2600 50  0001 C CNN
 F 3 "http://www.ti.com/lit/ds/symlink/lf357.pdf" H 6200 2700 50  0001 C CNN

Commit message: added some ordernr
Parts:
- J7: OrderNr S9337-ND -> 732-5315-ND (S9337-ND)
Changed lines of the file:
@@
 F 2 "Connector_PinHeader_2.54mm:PinHeader_1x02_P2.54mm_Vertical" H 4900 4750 50  0001 C CNN
 F 3 "~" H 4900 4750 50  0001 C CNN
-F 4 "S9337-ND " H 4900 4750 50  0001 C CNN "OrderNr"
+F 4 "732-5315-ND (S9337-ND)" H 4900 4750 50  0001 C CNN "OrderNr"
 	1    4900 4750
 	0    1    1    0

Commit message: I found a bug
Parts:
- C24: OrderN (none) -> 399-3684-6-ND
- J10, J5, J6, J8, J9: OrderN (none) -> S9337-ND
- J7: OrderN (none) -> 732-5315-ND (S9337-ND)
- R17, R18, R20, R22, R24: OrderN (none) -> 311-10.0KHRCT-ND
- R19, R21, R23: OrderN (none) -> 311-30.0KHRCT-ND
Changed lines of the file:
@@
 F 3 "~" H 3000 1100 50  0001 C CNN
 F 4 "399-3684-6-ND " H 3000 1100 50  0001 C CNN "OrderNr"
+F 5 "399-3684-6-ND " H 3000 1100 50  0001 C CNN "OrderN"
 	1    3000 1100
 	1    0    0    -1
@@
 F 2 "Resistor_SMD:R_0603_1608Metric" H 2550 1700 50  0001 C CNN
 F 3 "~" H 2550 1700 50  0001 C CNN
+F 4 " 311-10.0KHRCT-ND" H 2550 1700 50  0001 C CNN "OrderN"
 	1    2550 1700
 	1    0    0    -1
@@
 F 2 "Resistor_SMD:R_0603_1608Metric" H 6450 3000 50  0001 C CNN
 F 3 "~" H 6450 3000 50  0001 C CNN
+F 4 " 311-10.0KHRCT-ND" H 6450 3000 50  0001 C CNN "OrderN"
 	1    6450 3000
 	1    0    0    -1
@@
 F 2 "Resistor_SMD:R_0603_1608Metric" H 5450 2950 50  0001 C CNN
 F 3 "~" H 5450 2950 50  0001 C CNN
+F 4 "311-30.0KHRCT-ND " H 5450 2950 50  0001 C CNN "OrderN"
 	1    5450 2950
 	0    1    1    0
@@
 F 2 "Resistor_SMD:R_0603_1608Metric" H 5450 3700 50  0001 C CNN
 F 3 "~" H 5450 3700 50  0001 C CNN
+F 4 "311-30.0KHRCT-ND " H 5450 3700 50  0001 C CNN "OrderN"
 	1    5450 3700
 	0    1    1    0
@@
 F 2 "Resistor_SMD:R_0603_1608Metric" H 5450 2850 50  0001 C CNN
 F 3 "~" H 5450 2850 50  0001 C CNN
+F 4 " 311-10.0KHRCT-ND" H 5450 2850 50  0001 C CNN "OrderN"
 	1    5450 2850
 	0    -1   -1   0
@@
 F 2 "Resistor_SMD:R_0603_1608Metric" H 5450 3600 50  0001 C CNN
 F 3 "~" H 5450 3600 50  0001 C CNN
+F 4 " 311-10.0KHRCT-ND" H 5450 3600 50  0001 C CNN "OrderN"
 	1    5450 3600
 	0    -1   -1   0
@@
 F 3 "~" H 5100 4050 50  0001 C CNN
 F 4 "S9337-ND " H 5100 4050 50  0001 C CNN "OrderNr"
+F 5 "S9337-ND " H 5100 4050 50  0001 C CNN "OrderN"
 	1    5100 4050
 	0    1    1    0
@@
 F 3 "~" H 4900 4050 50  0001 C CNN
 F 4 "S9337-ND " H 4900 4050 50  0001 C CNN "OrderNr"
+F 5 "S9337-ND " H 4900 4050 50  0001 C CNN "OrderN"
 	1    4900 4050
 	0    1    1    0
@@
 F 3 "~" H 4900 4750 50  0001 C CNN
 F 4 "732-5315-ND (S9337-ND)" H 4900 4750 50  0001 C CNN "OrderNr"
+F 5 "732-5315-ND (S9337-ND)" H 4900 4750 50  0001 C CNN "OrderN"
 	1    4900 4750
 	0    1    1    0
@@
 F 3 "~" H 5100 4750 50  0001 C CNN
 F 4 "S9337-ND " H 5100 4750 50  0001 C CNN "OrderNr"
+F 5 "S9337-ND " H 5100 4750 50  0001 C CNN "OrderN"
 	1    5100 4750
 	0    1    1    0
@@
 F 2 "Resistor_SMD:R_0603_1608Metric" H 5450 4300 50  0001 C CNN
 F 3 "~" H 5450 4300 50  0001 C CNN
+F 4 " 311-10.0KHRCT-ND" H 5450 4300 50  0001 C CNN "OrderN"
 	1    5450 4300
 	0    -1   -1   0
@@
 F 2 "Resistor_SMD:R_0603_1608Metric" H 5450 4400 50  0001 C CNN
 F 3 "~" H 5450 4400 50  0001 C CNN
+F 4 "311-30.0KHRCT-ND " H 5450 4400 50  0001 C CNN "OrderN"
 	1    5450 4400
 	0    1    1    0
@@
 F 3 "~" H 5100 3300 50  0001 C CNN
 F 4 "S9337-ND " H 5100 3300 50  0001 C CNN "OrderNr"
+F 5 "S9337-ND " H 5100 3300 50  0001 C CNN "OrderN"
 	1    5100 3300
 	0    1    1    0
@@
 F 3 "~" H 4900 3300 50  0001 C CNN
 F 4 "S9337-ND " H 4900 3300 50  0001 C CNN "OrderNr"
+F 5 "S9337-ND " H 4900 3300 50  0001 C CNN "OrderN"
 	1    4900 3300
 	0    1    1    0
