File: Hardware/V1_0/MCU.sch (KiCad schematic (older format))
At the start: 1 part, among them U1 STM32F40X_LQFP64

Commit message: some work on the MCU part
Parts:
- added C10, C11, C12, C4, C5, C6, C8: 2.2u, Capacitor_SMD:C_0603_1608Metric, symbol Device:C_Small
- added C13, C9: 15p, Capacitor_SMD:C_0603_1608Metric, symbol Device:C_Small
- added C2, C3: 10uF, Capacitor_SMD:C_0805_2012Metric, symbol Device:C_Small
- added C7: 100n, Capacitor_SMD:C_0603_1608Metric, symbol Device:C_Small
- added J2: UART5, Connector_JST:JST_PH_B4B-PH-K_1x04_P2.00mm_Vertical, symbol Connector:Conn_01x04_Female
- added J3: USB_B_Mini, Connector_USB:USB_Mini-B_Lumberg_2486_01_Horizontal, symbol Connector:USB_B_Mini
- added J4: USART3_UART4, Connector_JST:JST_PH_B4B-PH-K_1x04_P2.00mm_Vertical, symbol Connector:Conn_01x04_Female
- added P1: SWD, Connector_JST:JST_PH_B6B-PH-K_1x06_P2.00mm_Vertical, symbol Connector:Conn_01x06_Female
- added R8, R9: 22R, Resistor_SMD:R_0603_1608Metric, symbol Device:R_Small
- added Y1: 8M, Crystal:Crystal_SMD_5032-4Pin_5.0x3.2mm, symbol Device:Crystal_GND24
Connections:
- net +3V3: now reaches U1.1 (VBAT)
- net +3V3: now also U1.19 (VDD), U1.32 (VDD), U1.48 (VDD), U1.64 (VDD), C10.1, C11.1, C12.1, C8.1, J2.4 (Pin_4), J4.4 (Pin_4), P1.6 (Pin_6)
- net GNDA: now reaches U1.12 (VSSA)
- net GNDA: now also C4.2
- net VREF: now reaches U1.13 (VDDA)
- net VREF: now also C4.1
- net GND: now reaches U1.18 (VSS)
- net GND: now also U1.28 (PB2-BOOT1), U1.63 (VSS), C10.2, C11.2, C12.2, C13.1, C5.1, C6.1, C7.2, C8.2, C9.1, J2.1 (Pin_1), J3.5 (GND), J3.6 (Shield), J4.1 (Pin_1), P1.4 (Pin_4), Y1.2, Y1.4
- net at U1.20 (PA4(ADC12_IN4/DAC1_OUT)): now also C3.1
- net at U1.21 (PA5(ADC12_IN5/DAC2_OUT)): now also C2.1
- net at U1.31 (VCAP1): now also C5.2
- net SDIO_D0: now reaches U1.38 (PC7)
- net SDIO_D1: now reaches U1.39 (PC8)
- net SDIO_D2: now reaches U1.40 (PC9)
- net USB_DM: now reaches U1.44 (PA11)
- net USB_DM: now also R9.2
- net USB_DP: now reaches U1.45 (PA12)
- net USB_DP: now also R8.2
- net SWDIO: now reaches U1.46 (PA13(JTMS-SWDIO))
- net SWDIO: now also P1.3 (Pin_3)
- net at U1.47 (VCAP2): now also C6.2
- net SWCLK: now reaches U1.49 (PA14(JTCK-SWCLK))
- net SWCLK: now also P1.5 (Pin_5)
- net at U1.5 (PH0-OSC_IN): now also C9.2, Y1.1
- net SDIO_D3: now reaches U1.51 (PC10)
- net SDIO_CK: now reaches U1.52 (PC11)
- net SDIO_DET: now reaches U1.53 (PC12)
- net SDIO_CMD: now reaches U1.54 (PD2)
- net at U1.6 (PH1-OSC_OUT): now also C13.2, Y1.3
- net BOOT0: now reaches U1.60 (BOOT0(VPP))
- net NRST: now reaches U1.7 (NRST)
- net NRST: now also C7.1, P1.2 (Pin_2)
- new net: J3.2 (D-), R9.1
- new net: J3.3 (D+), R8.1
- new net DAC1: C3.2
- new net DAC2: C2.2
- new net UART5_RX: J2.2 (Pin_2)
- new net UART5_TX: J2.3 (Pin_3)
- new net UART_RXD: J4.2 (Pin_2)
- new net UART_TXD: J4.3 (Pin_3)
- no-connect marks 0 -> 6
Other:
- note added: "Bypass, place next to VDD pins"
- note added: "Connected at power source\n"
- note added: "LQFP64\nTIM 2,3,4,5 PWM\n\n(TIM1 is more capable than TIM2 - 5\nTIM1 CH1 PIN 23 (N), 27(N), 34(N), 36(N), 41\nTIM1 CH2 PIN 42\nTIM1 CH3 PIN 43\nTIM1 CH4 PIN 44\n \n(Maybe prefer these ?) \nTIM2 CH1 PIN 14, 21\nTIM2 CH2 PIN 15, 55\nTIM2 CH3 PIN 16, 29\nTIM2 CH4 PIN 17, 30\n\nTIM3 CH1 PIN 37, 56\nTIM3 CH2 PIN 38 \nTIM3 CH3 PIN 26, 39\nTIM3 CH4 PIN 40 \n\nTIM4 CH1 PIN 58\nTIM4 CH2 PIN 59\nTIM4 CH3 P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"
- note added: "UART PINS \nUART4 TX: 14, 51\nUART4 RX: 15, 52 \nUART5 TX: 53\nUART5 RX: 54"

Commit message: tweaks
Connections:
- net +5V: now reaches J3.1 (VBUS)
- no-connect marks 6 -> 15
Other:
- note removed: "Connected at power source\n"
Changed lines of the file:
@@
 encoding utf-8
 Sheet 4 4
-Title ""
+Title "SYNTH"
 Date ""
-Rev ""
-Comp ""
+Rev "1"
+Comp "Bo Joel Svensson"
 Comment1 ""
 Comment2 ""
@@
 Wire Wire Line
 	6650 5450 6500 5450
-$Comp
-L power:GND #PWR015
-U 1 1 5E0B620C
-P 8300 5700
-F 0 "#PWR015" H 8300 5450 50  0001 C CNN
-F 1 "GND" H 8305 5527 50  0000 C CNN
-F 2 "" H 8300 5700 50  0001 C CNN
-F 3 "" H 8300 5700 50  0001 C CNN
-	1    8300 5700
-	1    0    0    -1
-$EndComp
-$Comp
-L power:GNDA #PWR016
-U 1 1 5E0B651C
-P 8800 5700
-F 0 "#PWR016" H 8800 5450 50  0001 C CNN
-F 1 "GNDA" H 8805 5527 50  0000 C CNN
-F 2 "" H 8800 5700 50  0001 C CNN
-F 3 "" H 8800 5700 50  0001 C CNN
-	1    8800 5700
-	1    0    0    -1
-$EndComp
-Text Notes 8450 6050 0    50   ~ 0
-Connected at power source\n
-$Comp
-L power:PWR_FLAG #FLG01
-U 1 1 5E0B7648
-P 8300 5550
-F 0 "#FLG01" H 8300 5625 50  0001 C CNN
-F 1 "PWR_FLAG" H 8300 5723 50  0000 C CNN
-F 2 "" H 8300 5550 50  0001 C CNN
-F 3 "~" H 8300 5550 50  0001 C CNN
-	1    8300 5550
-	1    0    0    -1
-$EndComp
-$Comp
-L power:PWR_FLAG #FLG02
-U 1 1 5E0B7923
-P 8800 5550
-F 0 "#FLG02" H 8800 5625 50  0001 C CNN
-F 1 "PWR_FLAG" H 8800 5723 50  0000 C CNN
-F 2 "" H 8800 5550 50  0001 C CNN
-F 3 "~" H 8800 5550 50  0001 C CNN
-	1    8800 5550
-	1    0    0    -1
-$EndComp
-Wire Wire Line
-	8300 5700 8300 5550
-Wire Wire Line
-	8800 5700 8800 5550
 Wire Wire Line
 	6250 4750 6250 4800
@@
 	6850 5250 6500 5250
 Connection ~ 6500 5250
+NoConn ~ 3550 1450
+NoConn ~ 3550 1550
+NoConn ~ 3550 1650
+NoConn ~ 3550 1750
+NoConn ~ 3550 2050
+NoConn ~ 3550 2150
+NoConn ~ 3550 2250
+NoConn ~ 3550 2350
+NoConn ~ 3550 2450
+$Comp
+L power:+5V #PWR0102
+U 1 1 5DD19B4C
+P 9850 3900
+F 0 "#PWR0102" H 9850 3750 50  0001 C CNN
+F 1 "+5V" H 9865 4073 50  0000 C CNN
+F 2 "" H 9850 3900 50  0001 C CNN
+F 3 "" H 9850 3900 50  0001 C CNN
+	1    9850 3900
+	1    0    0    -1
+$EndComp
+Wire Wire Line
+	9950 4050 9850 4050
+Wire Wire Line
+	9850 4050 9850 3900
 $EndSCHEMATC

Commit message: low energy work
Parts:
- renumbered C2 to C12, C3 to C13, C4 to C14, C5 to C15, C6 to C16, C7 to C17, C8 to C18, C9 to C19, C10 to C20, C11 to C21, C12 to C22, C13 to C23, R8 to R15, R9 to R16, U1 to U4
Connections:
- no-connect marks 15 -> 16

Commit message: update
Connections:
- net GNDA is gone; now on net GND: C14.2, U4.12 (VSSA)
- net DB0: now also U4.57 (PB5)
- net DB1: now also U4.58 (PB6)
- net DB2: now also U4.59 (PB7)
- net DB3: now also U4.61 (PB8)
- net DB4: now also U4.62 (PB9)
- net DB5: now also U4.29 (PB10)
- net DB6: now also U4.30 (PB11)
- net DB7: now also U4.33 (PB12)
- net N_LDAC_0: now reaches U4.10 (PC2(ADC123_IN12))
- net BUF_0: now reaches U4.11 (PC3(ADC123_IN13))
- net N_WR_0: now reaches U4.8 (PC0(ADC123_IN10))
- net N_CLR_0: now reaches U4.9 (PC1(ADC123_IN11))
- no-connect marks 16 -> 25
Changed lines of the file:
@@
 $EndComp
 $Comp
-L power:GND #PWR025
+L power:GND #PWR024
 U 1 1 5E0A2520
 P 7650 1400
-F 0 "#PWR025" H 7650 1150 50  0001 C CNN
+F 0 "#PWR024" H 7650 1150 50  0001 C CNN
 F 1 "GND" H 7650 1250 50  0000 C CNN
 F 2 "" H 7650 1400 60  0000 C CNN
@@
 	6600 1750 6850 1750
 $Comp
-L power:GND #PWR024
+L power:GND #PWR023
 U 1 1 5E0A254C
 P 7000 2050
-F 0 "#PWR024" H 7000 1800 50  0001 C CNN
+F 0 "#PWR023" H 7000 1800 50  0001 C CNN
 F 1 "GND" H 7000 1900 50  0000 C CNN
 F 2 "" H 7000 2050 60  0000 C CNN
@@
 	6050 2050 6250 2050
 $Comp
-L power:GND #PWR018
+L power:GND #PWR017
 U 1 1 5E0ADB29
 P 6300 2200
-F 0 "#PWR018" H 6300 1950 50  0001 C CNN
+F 0 "#PWR017" H 6300 1950 50  0001 C CNN
 F 1 "GND" H 6305 2027 50  0000 C CNN
 F 2 "" H 6300 2200 50  0001 C CNN
@@
 NoConn ~ 9850 2150
 $Comp
-L power:GND #PWR029
+L power:GND #PWR028
 U 1 1 56C1E83A
 P 9500 2200
-F 0 "#PWR029" H 9500 1950 50  0001 C CNN
+F 0 "#PWR028" H 9500 1950 50  0001 C CNN
 F 1 "GND" H 9500 2050 50  0000 C CNN
 F 2 "" H 9500 2200 60  0000 C CNN
@@
 $EndComp
 $Comp
-L power:GND #PWR021
+L power:GND #PWR020
 U 1 1 5A4BDE3D
 P 6550 2950
-F 0 "#PWR021" H 6550 2700 50  0001 C CNN
+F 0 "#PWR020" H 6550 2700 50  0001 C CNN
 F 1 "GND" H 6550 2800 50  0000 C CNN
 F 2 "" H 6550 2950 60  0000 C CNN
@@
 	6250 4250 6250 4350
 $Comp
-L power:GND #PWR020
+L power:GND #PWR019
 U 1 1 5A4BDE44
 P 6350 4400
-F 0 "#PWR020" H 6350 4150 50  0001 C CNN
+F 0 "#PWR019" H 6350 4150 50  0001 C CNN
 F 1 "GND" H 6350 4250 50  0000 C CNN
 F 2 "" H 6350 4400 60  0000 C CNN
@@
 	1    0    0    -1
 $EndComp
-$Comp
-L power:GNDA #PWR022
-U 1 1 5E0B57D1
-P 6650 5450
-F 0 "#PWR022" H 6650 5200 50  0001 C CNN
-F 1 "GNDA" H 6655 5277 50  0000 C CNN
-F 2 "" H 6650 5450 50  0001 C CNN
-F 3 "" H 6650 5450 50  0001 C CNN
-	1    6650 5450
-	1    0    0    -1
-$EndComp
 Wire Wire Line
 	6650 5450 6500 5450
@@
 	6250 4750 6250 4800
 $Comp
-L power:GND #PWR016
+L power:GND #PWR015
 U 1 1 5A4BDE3F
 P 6250 4800
-F 0 "#PWR016" H 6250 4550 50  0001 C CNN
+F 0 "#PWR015" H 6250 4550 50  0001 C CNN
 F 1 "GND" H 6250 4650 50  0000 C CNN
 F 2 "" H 6250 4800 60  0000 C CNN
@@
 	6250 4650 6250 4750
 $Comp
-L power:GND #PWR023
+L power:GND #PWR022
 U 1 1 5E0B842B
 P 6850 5950
-F 0 "#PWR023" H 6850 5700 50  0001 C CNN
+F 0 "#PWR022" H 6850 5700 50  0001 C CNN
 F 1 "GND" H 6850 5800 50  0000 C CNN
 F 2 "" H 6850 5950 60  0000 C CNN
@@
 $EndComp
 $Comp
-L power:GND #PWR031
+L power:GND #PWR030
 U 1 1 5AFF5692
 P 9800 2650
-F 0 "#PWR031" H 9800 2400 50  0001 C CNN
+F 0 "#PWR030" H 9800 2400 50  0001 C CNN
 F 1 "GND" H 9805 2477 50  0000 C CNN
 F 2 "" H 9800 2650 50  0001 C CNN
@@
 $EndComp
 $Comp
-L power:GND #PWR027
+L power:GND #PWR026
 U 1 1 5DDC5291
 P 8300 2650
-F 0 "#PWR027" H 8300 2400 50  0001 C CNN
+F 0 "#PWR026" H 8300 2400 50  0001 C CNN
 F 1 "GND" H 8305 2477 50  0000 C CNN
 F 2 "" H 8300 2650 50  0001 C CNN
@@
 UART_TXD
 $Comp
-L power:+3V3 #PWR030
+L power:+3V3 #PWR029
 U 1 1 5E094974
 P 9600 2900
-F 0 "#PWR030" H 9600 2750 50  0001 C CNN
+F 0 "#PWR029" H 9600 2750 50  0001 C CNN
 F 1 "+3V3" H 9615 3073 50  0000 C CNN
 F 2 "" H 9600 2900 50  0001 C CNN
@@
 $EndComp
 $Comp
-L power:+3V3 #PWR026
+L power:+3V3 #PWR025
 U 1 1 5E0CE9A4
 P 8100 2900
-F 0 "#PWR026" H 8100 2750 50  0001 C CNN
+F 0 "#PWR025" H 8100 2750 50  0001 C CNN
 F 1 "+3V3" H 8115 3073 50  0000 C CNN
 F 2 "" H 8100 2900 50  0001 C CNN
@@
 $EndComp
 $Comp
-L power:+3V3 #PWR028
+L power:+3V3 #PWR027
 U 1 1 5E0C17CE
 P 9500 1600
-F 0 "#PWR028" H 9500 1450 50  0001 C CNN
+F 0 "#PWR027" H 9500 1450 50  0001 C CNN
 F 1 "+3V3" H 9515 1773 50  0000 C CNN
 F 2 "" H 9500 1600 50  0001 C CNN
@@
 $EndComp
 $Comp
-L power:+3V3 #PWR017
+L power:+3V3 #PWR016
 U 1 1 5E0C1B22
 P 6250 5150
-F 0 "#PWR017" H 6250 5000 50  0001 C CNN
+F 0 "#PWR016" H 6250 5000 50  0001 C CNN
 F 1 "+3V3" H 6400 5200 50  0000 C CNN
 F 2 "" H 6250 5150 50  0001 C CNN
@@
 $EndComp
 $Comp
-L power:+3V3 #PWR019
+L power:+3V3 #PWR018
 U 1 1 5E0C23CE
 P 6300 3700
-F 0 "#PWR019" H 6300 3550 50  0001 C CNN
+F 0 "#PWR018" H 6300 3550 50  0001 C CNN
 F 1 "+3V3" H 6315 3873 50  0000 C CNN
 F 2 "" H 6300 3700 50  0001 C CNN
@@
 $EndComp
 $Comp
-L power:GND #PWR033
+L power:GND #PWR032
 U 1 1 5B04A901
 P 10350 4700
-F 0 "#PWR033" H 10350 4450 50  0001 C CNN
+F 0 "#PWR032" H 10350 4450 50  0001 C CNN
 F 1 "GND" H 10355 4527 50  0000 C CNN
 F 2 "" H 10350 4700 50  0001 C CNN
@@
 NoConn ~ 3550 2450
 $Comp
-L power:+5V #PWR032
+L power:+5V #PWR031
 U 1 1 5E0D79C8
 P 9850 3900
-F 0 "#PWR032" H 9850 3750 50  0001 C CNN
+F 0 "#PWR031" H 9850 3750 50  0001 C CNN
 F 1 "+5V" H 9865 4073 50  0000 C CNN
 F 2 "" H 9850 3900 50  0001 C CNN
@@
 	9850 4050 9850 3900
 NoConn ~ 3550 5550
-Text HLabel 2750 4100 0    50   Input ~ 0
-HBEN
-Text HLabel 2750 3700 0    50   Input ~ 0
+Text HLabel 3550 3750 0    50   Input ~ 0
 DB7
-Text HLabel 2750 4000 0    50   Input ~ 0
-NWR
-Text HLabel 2750 3200 0    50   Input ~ 0
+Text HLabel 3550 3250 0    50   Input ~ 0
 DB2
-Text HLabel 2750 3800 0    50   Input ~ 0
-NLDAC
-Text HLabel 2750 3500 0    50   Input ~ 0
+Text HLabel 3550 3550 0    50   Input ~ 0
 DB5
-Text HLabel 2750 3000 0    50   Input ~ 0
+Text HLabel 3550 3050 0    50   Input ~ 0
 DB0
-Text HLabel 2750 3300 0    50   Input ~ 0
+Text HLabel 3550 3350 0    50   Input ~ 0
 DB3
-Text HLabel 2750 3600 0    50   Input ~ 0
+Text HLabel 3550 3650 0    50   Input ~ 0
 DB6
-Text HLabel 2750 3100 0    50   Input ~ 0
+Text HLabel 3550 3150 0    50   Input ~ 0
 DB1
-Text HLabel 2750 3400 0    50   Input ~ 0
+Text HLabel 3550 3450 0    50   Input ~ 0
 DB4
-Text HLabel 2750 3900 0    50   Input ~ 0
-NCLR
-Text HLabel 2750 4300 0    50   Input ~ 0
-DMUX0
-Text HLabel 2750 4400 0    50   Input ~ 0
-DMUX1
+Text HLabel 3550 4350 0    50   Input ~ 0
+N_CLR_0
+Text HLabel 3550 4450 0    50   Input ~ 0
+N_LDAC_0
+Text HLabel 3550 4250 0    50   Input ~ 0
+N_WR_0
+Text HLabel 3550 4550 0    50   Input ~ 0
+BUF_0
+NoConn ~ 3550 2850
+NoConn ~ 3550 2950
+NoConn ~ 3550 3850
+NoConn ~ 3550 3950
+NoConn ~ 3550 4050
+NoConn ~ 3550 4650
+NoConn ~ 3550 4750
+NoConn ~ 3550 4850
+NoConn ~ 9950 4450
+$Comp
+L power:GND #PWR0101
+U 1 1 5E161FFD
+P 6650 5450
+F 0 "#PWR0101" H 6650 5200 50  0001 C CNN
+F 1 "GND" H 6650 5300 50  0000 C CNN
+F 2 "" H 6650 5450 60  0000 C CNN
+F 3 "" H 6650 5450 60  0000 C CNN
+	1    6650 5450
+	1    0    0    -1
+$EndComp
 $EndSCHEMATC

Commit message: experimenting
Parts:
- removed C12, C13: 10uF, Capacitor_SMD:C_0805_2012Metric, symbol Device:C_Small
- added D1: RED, LED_SMD:LED_0603_1608Metric, symbol Device:LED
- added D2: GREEN, LED_SMD:LED_0603_1608Metric, symbol Device:LED
- added R25, R26: 1k, Resistor_SMD:R_0603_1608Metric, symbol Device:R
- added RV1, RV2, RV3, RV4: R_POT, Potentiometer_THT:Potentiometer_Bourns_PTV09A-2_Single_Horizontal, symbol Device:R_POT
- J2: value UART5 -> USART2
- J4: value USART3_UART4 -> UART
Connections:
- net UART5_RX is gone; now on net USART2_RX: J2.2 (Pin_2)
- net UART5_TX is gone; now on net USART2_TX: J2.3 (Pin_3)
- net DAC1: now also U4.20 (PA4(ADC12_IN4/DAC1_OUT))
- net DAC2: now also U4.21 (PA5(ADC12_IN5/DAC2_OUT))
- net GND: now also D1.1 (K), D2.1 (K), RV1.3, RV2.3, RV3.3, RV4.3
- net UART_RXD: now also U4.15 (PA1(ADC123_IN1))
- net UART_TXD: now also U4.14 (PA0(ADC123_IN0/WKUP))
- net VREF: now also RV1.1, RV2.1, RV3.1, RV4.1
- net USART2_TX: now reaches U4.16 (PA2(ADC123_IN2))
- net USART2_RX: now reaches U4.17 (PA3(ADC123_IN3))
- net POT1: now reaches U4.22 (PA6(ADC12_IN6))
- net POT1: now also RV1.2
- net POT2: now reaches U4.23 (PA7(ADC12_IN7))
- net POT2: now also RV2.2
- net POT3: now reaches U4.24 (PC4(ADC12_IN14))
- net POT3: now also RV3.2
- net POT4: now reaches U4.25 (PC5(ADC12_IN15))
- net POT4: now also RV4.2
- net at U4.26 (PB0(ADC12_IN8)): now also R25.1
- net at U4.27 (PB1(ADC12_IN9)): now also R26.1
- new net: D1.2 (A), R25.2
- new net: D2.2 (A), R26.2
- no-connect marks 25 -> 15

Commit message: lots of tweaks
Parts:
- added SW3: BOOT0, Button_Switch_SMD:SW_SPDT_PCM12, symbol Switch:SW_SPDT
Connections:
- net +3V3: now also SW3.3 (C)
- net BOOT0: now also SW3.2 (B)
- net GND: now also SW3.1 (A)
Changed lines of the file:
@@
 Text Label 4250 6500 1    50   ~ 0
 POT4
+$Comp
+L Switch:SW_SPDT SW3
+U 1 1 5DDC212D
+P 1650 4600
+F 0 "SW3" H 1725 4425 50  0000 C CNN
+F 1 "BOOT0" H 1675 4800 50  0000 C CNN
+F 2 "Button_Switch_SMD:SW_SPDT_PCM12" H 1650 4600 50  0001 C CNN
+F 3 "~" H 1650 4600 50  0001 C CNN
+F 4 "401-2016-1-ND " H 1650 4600 50  0001 C CNN "OrderN"
+	1    1650 4600
+	0    1    1    0
+$EndComp
+$Comp
+L power:GND #PWR0139
+U 1 1 5DDC35F8
+P 1750 4900
+F 0 "#PWR0139" H 1750 4650 50  0001 C CNN
+F 1 "GND" H 1755 4727 50  0000 C CNN
+F 2 "" H 1750 4900 50  0001 C CNN
+F 3 "" H 1750 4900 50  0001 C CNN
+	1    1750 4900
+	1    0    0    -1
+$EndComp
+Wire Wire Line
+	1750 4800 1750 4900
+Text Label 1650 4100 0    50   ~ 0
+BOOT0
+Wire Wire Line
+	1650 4400 1650 4100
+Wire Wire Line
+	1550 4800 1550 4950
+Wire Wire Line
+	1550 4950 1100 4950
+Wire Wire Line
+	1100 4950 1100 4800
+$Comp
+L power:+3V3 #PWR?
+U 1 1 5E150BC4
+P 1100 4800
+F 0 "#PWR?" H 1100 4650 50  0001 C CNN
+F 1 "+3V3" H 1250 4850 50  0000 C CNN
+F 2 "" H 1100 4800 50  0001 C CNN
+F 3 "" H 1100 4800 50  0001 C CNN
+	1    1100 4800
+	1    0    0    -1
+$EndComp
 $EndSCHEMATC

Commit message: I found a bug
Parts:
- C14, C15, C16, C18, C20, C21, C22: OrderN 490-10731-1-ND -> 490-10731-1-ND
- U4: OrderN (none) -> 497-11767-ND
Changed lines of the file:
@@
 F 2 "Package_QFP:LQFP-64_10x10mm_P0.5mm" H 4800 3600 60  0001 C CNN
 F 3 "" H 4800 3600 60  0000 C CNN
+F 4 "497-11767-ND " H 4800 3600 50  0001 C CNN "OrderN"
 	1    4800 3600
 	1    0    0    -1
@@
 F 2 "Capacitor_SMD:C_0603_1608Metric" H 7338 3950 30  0001 C CNN
 F 3 "" H 7300 4100 60  0000 C CNN
-F 4 " 490-10731-1-ND " H 7300 4100 50  0001 C CNN "OrderN"
+F 4 "490-10731-1-ND" H 7300 4100 50  0001 C CNN "OrderN"
 	1    7300 4100
 	1    0    0    -1
@@
 F 2 "Capacitor_SMD:C_0603_1608Metric" H 6838 3950 30  0001 C CNN
 F 3 "" H 6800 4100 60  0000 C CNN
-F 4 " 490-10731-1-ND " H 6800 4100 50  0001 C CNN "OrderN"
+F 4 "490-10731-1-ND" H 6800 4100 50  0001 C CNN "OrderN"
 	1    6800 4100
 	1    0    0    -1
@@
 F 2 "Capacitor_SMD:C_0603_1608Metric" H 6588 3950 30  0001 C CNN
 F 3 "" H 6550 4100 60  0000 C CNN
-F 4 " 490-10731-1-ND " H 6550 4100 50  0001 C CNN "OrderN"
+F 4 "490-10731-1-ND" H 6550 4100 50  0001 C CNN "OrderN"
 	1    6550 4100
 	1    0    0    -1
@@
 F 2 "Capacitor_SMD:C_0603_1608Metric" H 7088 3950 30  0001 C CNN
 F 3 "" H 7050 4100 60  0000 C CNN
-F 4 " 490-10731-1-ND " H 7050 4100 50  0001 C CNN "OrderN"
+F 4 "490-10731-1-ND" H 7050 4100 50  0001 C CNN "OrderN"
 	1    7050 4100
 	1    0    0    -1
@@
 F 2 "Capacitor_SMD:C_0603_1608Metric" H 6538 5200 30  0001 C CNN
 F 3 "" H 6500 5350 60  0000 C CNN
-F 4 " 490-10731-1-ND " H 6500 5350 50  0001 C CNN "OrderN"
+F 4 "490-10731-1-ND" H 6500 5350 50  0001 C CNN "OrderN"
 	1    6500 5350
 	1    0    0    -1
@@
 F 2 "Capacitor_SMD:C_0603_1608Metric" H 6538 5650 30  0001 C CNN
 F 3 "" H 6500 5800 60  0000 C CNN
-F 4 " 490-10731-1-ND " H 6500 5800 50  0001 C CNN "OrderN"
+F 4 "490-10731-1-ND" H 6500 5800 50  0001 C CNN "OrderN"
 	1    6500 5800
 	0    1    1    0
@@
 F 2 "Capacitor_SMD:C_0603_1608Metric" H 6538 5900 30  0001 C CNN
 F 3 "" H 6500 6050 60  0000 C CNN
-F 4 " 490-10731-1-ND " H 6500 6050 50  0001 C CNN "OrderN"
+F 4 "490-10731-1-ND" H 6500 6050 50  0001 C CNN "OrderN"
 	1    6500 6050
 	0    1    1    0
